File: Eagle/main.brd (EAGLE design)
At the start: 304.8 x 254 mm, 170 parts, among them M041C 74HC00D, M085C 74HC00D, M0FA30 74HC00D, M0FA31 74HC00D, M0FA40 74HC00D, M0FA41 74HC00D, M0FA50 74HC00D, M0FA51 74HC00D, M0FA60 74HC00D, M0FA61 74HC00D, M0FA70 74HC00D, M0FA71 74HC00D, M0FA80 74HC00D, M0FA81 74HC00D, M0HA0 74HC00D, M0HA1 74HC00D, M0HA2 74HC00D, M120C 74HC00D, M163C 74HC00D, M197C 74HC00D, M1FA10 74HC00D, M1FA11 74HC00D, M1FA20 74HC00D, M1FA21 74HC00D, M1FA30 74HC00D, M1FA31 74HC00D, M1FA40 74HC00D, M1FA41 74HC00D, M1FA50 74HC00D, M1FA51 74HC00D, M1FA60 74HC00D, M1FA61 74HC00D, M1FA70 74HC00D, M1FA71 74HC00D, M1FA80 74HC00D, M1FA81 74HC00D, M1FA90 74HC00D, M1FA91 74HC00D, M1HA0 74HC00D, M241C 74HC00D, M285C 74HC00D, M2FA00 74HC00D, M2FA01 74HC00D, M2HA1 74HC00D, M2HA2 74HC00D, M2HA3 74HC00D, M2HA4 74HC00D, M2HA5 74HC00D, M2HA6 74HC00D, M2HA7 74HC00D, M2HA8 74HC00D

Commit message: SystemVerilog with assigns
Parts:
- removed BEL7, BENC0, BENC10, BENC1_1, BENC2, BENC3, BENC4, BENC5, BENC6, BENC7, BENC8, BENC9, BSEL0, BSEL1, BSEL10, BSEL11, BSEL12, BSEL13, BSEL14, BSEL15, BSEL16, BSEL17, BSEL18, BSEL19, BSEL2, BSEL20, BSEL21, BSEL22, BSEL23, BSEL24, BSEL25, BSEL26, BSEL27, BSEL28, BSEL29, BSEL3, BSEL30, BSEL31, BSEL32, BSEL33, BSEL34, BSEL35, BSEL36, BSEL37, BSEL38, BSEL39, BSEL4, BSEL40, BSEL41, BSEL42, BSEL43, BSEL44, BSEL45, BSEL46, BSEL47, BSEL5, BSEL58, BSEL59, BSEL6, BSEL60, BSEL61, BSEL62, BSEL63, BSEL64, BSEL65, BSEL66, BSEL67, BSEL68, BSEL69, BSEL70, BSEL71, BSEL8, BSEL9, CLA0, CLA1, CLA100, CLA101, CLA110, CLA111, CLA120, CLA121, CLA130, CLA131, CLA140, CLA141, CLA150, CLA151, CLA20, CLA21, CLA30, CLA31, CLA40, CLA41, CLA50, CLA51, CLA6, CLA70, CLA71, CLA80, CLA81, CLA90, CLA91, CLAP0, CLAP1, CLAP2, CLAP3, CLAP4, CLAP5, CLAP6, CLAP7, CLAP8, CLU0, CLU1, CLU2, CLU3, CLU4, CLU5, CLU6, HA1B0, M041C, M085C, M0FA30, M0FA31, M0FA40, M0FA41, M0FA50, M0FA51, M0FA60, M0FA61, M0FA70, M0FA71, M0FA80, M0FA81, M0HA0, M0HA1, M0HA2, M120C, M163C, M197C, M1FA10, M1FA11, M1FA20, M1FA21, M1FA30, M1FA31, M1FA40, M1FA41, M1FA50, M1FA51, M1FA60, M1FA61, M1FA70, M1FA71, M1FA80, M1FA81, M1FA90, M1FA91, M1HA0, M241C, M285C, M2FA00, M2FA01, M2HA1, M2HA2, M2HA3, M2HA4, M2HA5, M2HA6, M2HA7, M2HA8: 74HC00D, 74HC00:SO14
- added IC1, IC10, IC100, IC101, IC102, IC103, IC104, IC105, IC106, IC107, IC108, IC109, IC11, IC110, IC111, IC112, IC113, IC114, IC115, IC116, IC117, IC118, IC119, IC12, IC120, IC121, IC122, IC123, IC124, IC125, IC126, IC127, IC128, IC129, IC13, IC130, IC131, IC132, IC133, IC134, IC135, IC136, IC137, IC138, IC139, IC14, IC140, IC141, IC142, IC143, IC144, IC145, IC146, IC147, IC148, IC149, IC15, IC150, IC151, IC152, IC153, IC154, IC155, IC156, IC157, IC158, IC159, IC16, IC160, IC161, IC162, IC163, IC164, IC165, IC166, IC167, IC168, IC169, IC17, IC170, IC171, IC172, IC173, IC174, IC175, IC176, IC177, IC178, IC179, IC18, IC180, IC181, IC182, IC183, IC184, IC185, IC186, IC187, IC188, IC189, IC19, IC190, IC191, IC192, IC193, IC194, IC195, IC196, IC197, IC198, IC199, IC2, IC20, IC200, IC201, IC202, IC203, IC204, IC205, IC206, IC207, IC208, IC209, IC21, IC210, IC211, IC212, IC213, IC214, IC215, IC216, IC217, IC218, IC219, IC22, IC220, IC221, IC222, IC223, IC224, IC225, IC226, IC227, IC228, IC229, IC23, IC230, IC231, IC232, IC233, IC234, IC235, IC236, IC237, IC238, IC239, IC24, IC240, IC241, IC242, IC243, IC244, IC245, IC246, IC247, IC248, IC249, IC25, IC250, IC251, IC252, IC253, IC254, IC255, IC256, IC257, IC258, IC259, IC26, IC260, IC261, IC262, IC263, IC264, IC265, IC266, IC267, IC268, IC269, IC27, IC270, IC271, IC272, IC273, IC274, IC275, IC276, IC277, IC278, IC279, IC28, IC280, IC281, IC282, IC283, IC284, IC285, IC286, IC287, IC288, IC289, IC29, IC290, IC291, IC292, IC293, IC294, IC295, IC296, IC297, IC298, IC299, IC3, IC30, IC300, IC301, IC302, IC303, IC304, IC305, IC306, IC307, IC308, IC309, IC31, IC310, IC311, IC312, IC313, IC314, IC315, IC316, IC317, IC318, IC319, IC32, IC320, IC321, IC322, IC323, IC324, IC325, IC326, IC327, IC328, IC329, IC33, IC330, IC331, IC332, IC333, IC34, IC35, IC352, IC353, IC354, IC355, IC356, IC357, IC358, IC359, IC36, IC360, IC361, IC362, IC363, IC364, IC365, IC366, IC367, IC368, IC369, IC37, IC370, IC371, IC38, IC39, IC4, IC40, IC41, IC42, IC43, IC44, IC45, IC46, IC47, IC48, IC49, IC5, IC50, IC51, IC52, IC53, IC54, IC55, IC56, IC57, IC58, IC59, IC6, IC60, IC61, IC62, IC63, IC64, IC65, IC66, IC67, IC68, IC69, IC7, IC70, IC71, IC72, IC73, IC74, IC75, IC76, IC77, IC78, IC79, IC8, IC80, IC81, IC82, IC83, IC84, IC85, IC86, IC87, IC88, IC89, IC9, IC90, IC91, IC92, IC93, IC94, IC95, IC96, IC97, IC98, IC99: 74HC00D, 74HC00:SO14
- added IC334, IC335, IC336, IC337, IC338, IC339, IC340, IC341, IC342, IC343, IC344, IC345, IC346, IC347, IC348, IC349, IC350, IC351: 74HC377DW, 74HC00:SO20W
- added LED1, LED2: (no value), led:LED5MM
- added R1, R2: 22k, resistor:0207/10
- added X1, X2: 2534-5, con-3m:PAK100/2500-5-34
Connections:
- removed net A0: BEL7.10, BENC0.1, BENC0.2, BSEL0.10, BSEL1.5, BSEL2.13, BSEL2.2, BSEL66.5, BSEL8.5, BSEL9.13, BSEL9.2
- removed net A1: BENC0.12, BENC0.5, BENC1_1.1, BENC2.10, BENC2.9, BSEL10.13, BSEL10.5, BSEL11.13, BSEL11.5, BSEL12.13, BSEL12.2, BSEL13.13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
- removed net A2: BENC0.13, BENC1_1.5, BENC2.12, BENC2.13
- removed net A3: BENC2.1, BENC2.2, BENC3.10, BENC4.1, BENC4.4, BENC6.1, BENC6.2, BSEL17.13, BSEL17.5, BSEL18.13, BSEL18.5, BSEL19.13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
- removed net A4: BENC4.10, BENC4.2, BENC5.12, BENC5.13
- removed net A5: BENC5.4, BENC5.5, BENC6.13, BENC7.4, BENC7.9, BENC9.4, BENC9.5, BSEL31.13, BSEL31.5, BSEL32.13, BSEL32.5, BSEL33.13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
- removed net A6: BENC7.10, BENC8.2, BENC9.1, BENC9.2
- removed net A7: BENC10.5, BENC8.10, BENC8.9, BSEL45.13, BSEL45.5, BSEL46.13, BSEL46.5, BSEL47.13, BSEL47.2, BSEL58.13, BSEL58.2, BSEL62.13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
- removed net B0: BSEL23.9, BSEL37.9, BSEL61.9, BSEL66.4, BSEL66.9, BSEL67.4, BSEL67.9, BSEL9.9
- removed net B1: BSEL22.12, BSEL23.12, BSEL36.12, BSEL37.12, BSEL60.12, BSEL61.12, BSEL8.12, BSEL9.12
- removed net B2: BSEL22.1, BSEL23.1, BSEL36.1, BSEL37.1, BSEL60.1, BSEL61.1, BSEL8.1, BSEL9.1
- removed net B3: BEL7.4, BSEL21.4, BSEL22.4, BSEL35.4, BSEL36.4, BSEL59.4, BSEL60.4, BSEL8.4
- removed net B4: BEL7.9, BSEL16.9, BSEL2.9, BSEL21.9, BSEL30.9, BSEL35.9, BSEL44.9, BSEL59.9
- removed net B5: BSEL1.12, BSEL15.12, BSEL16.12, BSEL2.12, BSEL29.12, BSEL30.12, BSEL43.12, BSEL44.12
- removed net B6: BSEL1.1, BSEL15.1, BSEL16.1, BSEL2.1, BSEL29.1, BSEL30.1, BSEL43.1, BSEL44.1
- removed net B7: BSEL0.4, BSEL0.9, BSEL1.4, BSEL14.4, BSEL14.9, BSEL15.4, BSEL28.4, BSEL28.9, BSEL29.4, BSEL42.4, BSEL42.9, BSEL43.4
- removed net PP2_SE_N: HA1B0.3
- removed net Z10: M2HA8.10, M2HA8.5
- new net ADD_C0: IC192.11, IC199.2, IC199.5, IC222.1
- new net ADD_G_N0: IC195.12, IC195.3, IC195.4, IC222.5
- new net ADD_G_N1: IC196.12, IC196.3, IC196.4, IC222.13
- new net ADD_G_N2: IC197.12, IC197.3, IC197.4, IC223.5
- new net ADD_G_N3: IC205.12, IC205.3, IC205.4, IC223.13
- new net ADD_G_N4: IC210.12, IC210.3, IC210.4, IC224.5
- new net ADD_G_N5: IC211.12, IC211.3, IC211.4, IC224.13
- new net ADD_G_N6: IC212.12, IC212.3, IC212.4, IC225.5
- new net ADD_G_N7: IC220.12, IC220.3, IC220.4, IC225.13
- new net ADD_P0: IC198.8, IC222.2
- new net ADD_P1: IC200.6, IC222.10
- new net ADD_P2: IC203.3, IC223.2
- new net ADD_P3: IC203.11, IC223.10
- new net ADD_P4: IC213.8, IC224.2
- new net ADD_P5: IC215.6, IC224.10
- new net ADD_P6: IC218.3, IC225.2
- new net ADD_P7: IC218.11, IC225.10
- new net AND0: IC171.6, IC244.5
- new net AND1: IC171.11, IC247.5
- new net AND2: IC172.6, IC251.2
- new net AND3: IC172.11, IC254.2
- new net AND4: IC173.6, IC256.2
- new net AND5: IC173.11, IC265.2
- new net AND6: IC174.6, IC267.2
- new net AND7: IC174.11, IC270.2
- new net AOP: IC242.3, IC244.4, IC247.4, IC251.1, IC254.1, IC256.1, IC265.1, IC267.1, IC270.1
- new net AREG0: IC243.5
- new net AREG1: IC249.2, IC263.3
- new net AREG2: IC253.2, IC263.11
- new net AREG3: IC253.13
- new net AREG4: IC258.10
- new net AREG5: IC259.5
- new net AREG6: IC269.2
- new net AREG7: IC269.13
- new net AWE: IC239.11
- new net A_MULT0: IC1.1, IC1.2, IC13.10, IC14.5, IC17.13, IC17.2, IC20.10, IC21.5, IC24.13, IC24.2, IC69.2, X1.3
- new net A_MULT1: IC1.12, IC1.5, IC12.2, IC12.5, IC126.2, IC126.5, IC15.2, IC15.5, IC16.2, IC16.5, IC18.2, IC18.5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
- new net A_MULT2: IC1.13, IC2.2, IC3.12, IC3.13, X1.7
- new net A_MULT3: IC154.10, IC154.9, IC157.2, IC157.5, IC26.2, IC26.5, IC29.2, IC29.5, IC3.1, IC3.2, IC30.2, IC30.5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
- new net A_MULT4: IC5.2, IC5.5, IC7.12, IC7.13, X1.11
- new net A_MULT5: IC10.4, IC10.5, IC114.2, IC114.5, IC40.2, IC40.5, IC43.2, IC43.5, IC44.2, IC44.5, IC46.2, IC46.5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
- new net A_MULT6: IC10.1, IC10.2, IC8.5, IC9.2, X1.15
- new net A_MULT7: IC108.2, IC108.5, IC11.5, IC54.2, IC54.5, IC57.2, IC57.5, IC58.2, IC58.5, IC60.2, IC60.5, IC61.2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
- new net A_VOP0: IC171.1, IC175.1, IC175.2, IC177.1, IC177.2, IC183.1, IC183.13, IC195.2, IC195.5, IC198.4, IC198.5, IC263.10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
- new net A_VOP1: IC171.9, IC175.4, IC175.5, IC177.10, IC177.9, IC184.1, IC184.13, IC196.2, IC196.5, IC198.12, IC198.13, X2.5
- new net A_VOP2: IC172.1, IC175.10, IC175.9, IC178.1, IC178.2, IC185.1, IC185.13, IC197.2, IC197.5, IC200.10, IC200.9, X2.7
- new net A_VOP3: IC172.9, IC175.12, IC175.13, IC178.10, IC178.9, IC186.1, IC186.13, IC203.4, IC203.5, IC205.2, IC205.5, X2.9
- new net A_VOP4: IC173.1, IC176.1, IC176.2, IC179.1, IC179.2, IC187.1, IC187.13, IC210.2, IC210.5, IC213.4, IC213.5, X2.11
- new net A_VOP5: IC173.9, IC176.4, IC176.5, IC179.10, IC179.9, IC188.1, IC188.13, IC211.2, IC211.5, IC213.12, IC213.13, X2.13
- new net A_VOP6: IC174.1, IC176.10, IC176.9, IC180.1, IC180.2, IC189.1, IC189.13, IC212.2, IC212.5, IC215.10, IC215.9, X2.15
- new net A_VOP7: IC174.9, IC176.12, IC176.13, IC180.10, IC180.9, IC190.1, IC190.13, IC218.4, IC218.5, IC220.2, IC220.5, X2.17
- new net BOP: IC242.6, IC244.1, IC247.1, IC251.4, IC254.4, IC256.4, IC265.4, IC267.4, IC270.4
- new net B_MULT0: IC24.9, IC38.9, IC52.9, IC66.9, IC69.1, IC69.12, IC72.4, IC72.9, X1.19
- new net B_MULT1: IC21.12, IC24.12, IC35.12, IC38.12, IC49.12, IC52.12, IC63.12, IC66.12, X1.21
- new net B_MULT2: IC21.1, IC24.1, IC35.1, IC38.1, IC49.1, IC52.1, IC63.1, IC66.1, X1.23
- new net B_MULT3: IC20.4, IC21.4, IC34.4, IC35.4, IC48.4, IC49.4, IC62.4, IC63.4, X1.25
- new net B_MULT4: IC17.9, IC20.9, IC31.9, IC34.9, IC45.9, IC48.9, IC59.9, IC62.9, X1.27
- new net B_MULT5: IC14.12, IC17.12, IC28.12, IC31.12, IC42.12, IC45.12, IC56.12, IC59.12, X1.29
- new net B_MULT6: IC14.1, IC17.1, IC28.1, IC31.1, IC42.1, IC45.1, IC56.1, IC59.1, X1.31
- new net B_MULT7: IC13.4, IC13.9, IC14.4, IC27.4, IC27.9, IC28.4, IC41.4, IC41.9, IC42.4, IC55.4, IC55.9, IC56.4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
- new net B_VOP0: IC171.2, IC177.4, IC177.5, IC183.2, IC183.5, IC191.2, IC191.5, X2.19
- new net B_VOP1: IC171.10, IC177.12, IC177.13, IC184.2, IC184.5, IC193.2, IC193.5, X2.21
- new net B_VOP2: IC172.2, IC178.4, IC178.5, IC185.2, IC185.5, IC194.2, IC194.5, X2.23
- new net B_VOP3: IC172.10, IC178.12, IC178.13, IC186.2, IC186.5, IC204.2, IC204.5, X2.25
- new net B_VOP4: IC173.2, IC179.4, IC179.5, IC187.2, IC187.5, IC207.2, IC207.5, X2.27
- new net B_VOP5: IC173.10, IC179.12, IC179.13, IC188.2, IC188.5, IC208.2, IC208.5, X2.29
- new net B_VOP6: IC174.2, IC180.4, IC180.5, IC189.2, IC189.5, IC209.2, IC209.5, X2.31
- new net B_VOP7: IC174.10, IC180.12, IC180.13, IC190.2, IC190.5, IC219.2, IC219.5, X2.33
- new net CCLEAR: X2.22
- new net CIN: IC192.9
- new net CIN1: IC201.2, IC201.5, IC222.6, IC222.9
- new net CIN2: IC202.2, IC202.5, IC222.11, IC223.1
- new net CIN3: IC206.2, IC206.5, IC223.6, IC223.9
- new net CIN4: IC214.2, IC214.5, IC223.11, IC224.1
- new net CIN5: IC216.2, IC216.5, IC224.6, IC224.9
- new net CIN6: IC217.2, IC217.5, IC224.11, IC225.1
- new net CIN7: IC221.2, IC221.5, IC225.6, IC225.9
- new net CLK: X2.20
- new net CLK3: IC334.11, IC335.11
- new net COP: IC242.8, IC245.1, IC248.1, IC252.1, IC255.1, IC257.1, IC266.1, IC268.1, IC271.1
- new net COUT: IC225.11
- new net CSEL: IC192.1, IC192.10, IC192.2, X2.24
- new net DOP: IC242.11, IC245.4, IC248.4, IC252.4, IC255.4, IC257.4, IC266.4, IC268.4, IC271.4
- new net EOP: IC243.3, IC246.1, IC250.12, IC260.12, IC261.12, IC262.12, IC272.12, IC273.12, IC274.12
- new net FOP: IC239.8, IC243.4, IC249.1, IC253.1, IC253.12, IC258.9, IC259.4, IC269.1, IC269.12
- new net GND1: IC171.7, IC172.7, IC173.7, IC174.7, IC175.7, IC176.7, IC177.7, IC178.7, IC179.7, IC180.7, IC181.7, IC182.7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
- new net GND3: IC275.7, IC276.7, IC277.7, IC278.7, IC279.7, IC280.7, IC281.7, IC282.7, IC283.7, IC284.7, IC285.7, IC286.7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
- new net INST4: IC360.1, IC361.1, IC363.1, IC364.1, IC365.1, IC366.1, IC367.1, IC370.12, IC370.13
- new net INST4N: IC352.1, IC353.1, IC354.1, IC355.1, IC356.1, IC357.1, IC358.1, IC359.1, IC370.11
- new net INST5: IC354.9, IC355.9, IC356.2, IC357.2, IC358.2, IC358.9, IC359.2, IC359.9, IC363.9, IC364.2, IC365.2, IC366.2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
- new net INST5N: IC352.2, IC352.9, IC353.2, IC353.9, IC354.2, IC355.2, IC356.9, IC357.9, IC360.2, IC360.9, IC361.2, IC361.9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
- new net INST6: IC371.4, IC371.5
- new net INST6N: IC371.6
- new net INST7: IC353.10, IC355.10, IC357.10, IC359.10, IC361.10, IC363.10, IC365.10, IC367.10, IC371.1, IC371.2
- new net INST7N: IC352.10, IC354.10, IC356.10, IC358.10, IC360.10, IC364.10, IC366.10, IC371.3
- new net MPROD10: IC346.7
- new net MPROD11: IC346.8
- new net MPROD12: IC346.13
- new net MPROD13: IC346.14
- new net MPROD14: IC346.17
- new net MPROD15: IC346.18
- new net MPROD8: IC346.3
- new net MPROD9: IC346.4
- new net N$1007: IC283.6, IC283.9
- new net N$1008: IC283.10, IC283.11
- new net N$1009: IC288.10, IC288.11
- new net N$1010: IC288.6, IC288.9
- new net N$1011: IC288.8, IC291.1, IC291.13
- new net N$1012: IC291.12, IC291.3, IC291.4
- new net N$1013: IC291.6, IC291.9
- new net N$1014: IC291.10, IC291.11
- new net N$1015: IC286.12, IC286.3, IC286.4
- new net N$1016: IC282.8, IC286.1, IC286.13
- new net N$1017: IC286.10, IC286.11
- new net N$1018: IC286.6, IC286.9
- new net N$1019: IC282.10, IC282.11
- new net N$1020: IC282.6, IC282.9
- new net N$1021: IC287.6, IC287.9
- new net N$1022: IC287.10, IC287.11
- new net N$1023: IC287.8, IC290.1, IC290.13
- new net N$1024: IC290.12, IC290.3, IC290.4
- new net N$1025: IC290.6, IC290.9
- new net N$1026: IC290.10, IC290.11
- new net N$1027: IC284.3, IC284.9
- new net N$1028: IC284.10, IC284.6
- new net N$1029: IC289.3, IC289.5
- new net N$1030: IC284.11, IC289.4
- new net N$1031: IC285.2, IC289.11
- new net N$1032: IC285.1, IC289.8
- new net N$1033: IC285.13, IC285.8
- new net N$1034: IC285.12, IC285.6
- new net N$1035: IC298.6, IC298.9
- new net N$1036: IC298.10, IC298.11
- new net N$1037: IC298.12, IC298.3, IC298.4
- new net N$1038: IC294.8, IC298.1, IC298.13
- new net N$1039: IC294.6, IC294.9
- new net N$1040: IC294.10, IC294.11
- new net N$1041: IC300.10, IC300.11
- new net N$1042: IC300.6, IC300.9
- new net N$1043: IC300.8, IC303.1, IC303.13
- new net N$1044: IC303.12, IC303.3, IC303.4
- new net N$1045: IC303.6, IC303.9
- new net N$1046: IC303.10, IC303.11
- new net N$1047: IC297.12, IC297.3, IC297.4
- new net N$1048: IC293.8, IC297.1, IC297.13
- new net N$1049: IC297.10, IC297.11
- new net N$1050: IC297.6, IC297.9
- new net N$1051: IC293.10, IC293.11
- new net N$1052: IC293.6, IC293.9
- new net N$1053: IC299.6, IC299.9
- new net N$1054: IC299.10, IC299.11
- new net N$1055: IC299.8, IC302.1, IC302.13
- new net N$1056: IC302.12, IC302.3, IC302.4
- new net N$1057: IC302.6, IC302.9
- new net N$1058: IC302.10, IC302.11
- new net N$1059: IC295.3, IC295.9
- new net N$1060: IC295.10, IC295.6
- new net N$1061: IC301.3, IC301.5
- new net N$1062: IC295.11, IC301.4
- new net N$1063: IC296.2, IC301.11
- new net N$1064: IC296.1, IC301.8
- new net N$1065: IC296.13, IC296.8
- new net N$1066: IC296.12, IC296.6
- new net N$1067: IC309.6, IC309.9
- new net N$1068: IC309.10, IC309.11
- new net N$1069: IC309.12, IC309.3, IC309.4
- new net N$1070: IC305.8, IC309.1, IC309.13
- new net N$1071: IC305.6, IC305.9
- new net N$1072: IC305.10, IC305.11
- new net N$1073: IC311.10, IC311.11
- new net N$1074: IC311.6, IC311.9
- new net N$1075: IC311.8, IC314.1, IC314.13
- new net N$1076: IC314.12, IC314.3, IC314.4
- new net N$1077: IC314.6, IC314.9
- new net N$1078: IC314.10, IC314.11
- new net N$1079: IC308.12, IC308.3, IC308.4
- new net N$1080: IC304.8, IC308.1, IC308.13
- new net N$1081: IC308.10, IC308.11
- new net N$1082: IC308.6, IC308.9
- new net N$1083: IC304.10, IC304.11
- new net N$1084: IC304.6, IC304.9
- new net N$1085: IC310.6, IC310.9
- new net N$1086: IC310.10, IC310.11
- new net N$1087: IC310.8, IC313.1, IC313.13
- new net N$1088: IC313.12, IC313.3, IC313.4
- new net N$1089: IC313.6, IC313.9
- new net N$1090: IC313.10, IC313.11
- new net N$1091: IC306.3, IC306.9
- new net N$1092: IC306.10, IC306.6
- new net N$1093: IC312.3, IC312.5
- new net N$1094: IC306.11, IC312.4
- new net N$1095: IC307.2, IC312.11
- new net N$1096: IC307.1, IC312.8
- new net N$1097: IC307.13, IC307.8
- new net N$1098: IC307.12, IC307.6
- new net N$1099: IC320.6, IC320.9
- new net N$1100: IC320.10, IC320.11
- new net N$1101: IC320.12, IC320.3, IC320.4
- new net N$1102: IC316.8, IC320.1, IC320.13
- new net N$1103: IC316.6, IC316.9
- new net N$1104: IC316.10, IC316.11
- new net N$1105: IC322.10, IC322.11
- new net N$1106: IC322.6, IC322.9
- new net N$1107: IC322.8, IC325.1, IC325.13
- new net N$1108: IC325.12, IC325.3, IC325.4
- new net N$1109: IC325.6, IC325.9
- new net N$1110: IC325.10, IC325.11
- new net N$1111: IC319.12, IC319.3, IC319.4
- new net N$1112: IC315.8, IC319.1, IC319.13
- new net N$1113: IC319.10, IC319.11
- new net N$1114: IC319.6, IC319.9
- new net N$1115: IC315.10, IC315.11
- new net N$1116: IC315.6, IC315.9
- new net N$1117: IC321.6, IC321.9
- new net N$1118: IC321.10, IC321.11
- new net N$1119: IC321.8, IC324.1, IC324.13
- new net N$1120: IC324.12, IC324.3, IC324.4
- new net N$1121: IC324.6, IC324.9
- new net N$1122: IC324.10, IC324.11
- new net N$1123: IC317.3, IC317.9
- new net N$1124: IC317.10, IC317.6
- new net N$1125: IC323.3, IC323.5
- new net N$1126: IC317.11, IC323.4
- new net N$1127: IC318.2, IC323.11
- new net N$1128: IC318.1, IC323.8
- new net N$1132: IC326.6, IC326.9
- new net N$1133: IC326.11, IC328.1
- new net N$1134: IC328.6, IC328.9
- new net N$1135: IC327.1, IC328.11
- new net N$1136: IC327.6, IC327.9
- new net N$1137: IC327.11, IC329.1
- new net N$1138: IC329.6, IC329.9
- new net N$1139: IC329.11, IC330.2
- new net N$1140: IC330.6, IC330.9
- new net N$1141: IC330.11, IC333.1
- new net N$1142: IC333.6, IC333.9
- new net N$1143: IC332.1, IC333.11
- new net N$1144: IC332.6, IC332.9
- new net N$1145: IC331.1, IC332.11
- new net N$1146: IC363.3, IC363.4, IC363.5
- new net N$1147: IC363.12, IC363.13, IC363.8
- new net N$1152: IC363.6, IC369.9
- new net N$1153: IC363.11, IC369.10
- new net N$503: LED1.A, R1.1
- new net N$507: LED2.A, R2.1
- new net N$509: IC171.3, IC171.4, IC171.5
- new net N$511: IC171.12, IC171.13, IC171.8
- new net N$513: IC172.3, IC172.4, IC172.5
- new net N$514: IC172.12, IC172.13, IC172.8
- new net N$516: IC173.3, IC173.4, IC173.5
- new net N$518: IC173.12, IC173.13, IC173.8
- new net N$520: IC174.3, IC174.4, IC174.5
- new net N$522: IC174.12, IC174.13, IC174.8
- new net N$524: IC177.3, IC181.1
- new net N$526: IC177.6, IC181.2
- new net N$529: IC177.8, IC181.4
- new net N$530: IC177.11, IC181.5
- new net N$531: IC178.3, IC181.9
- new net N$533: IC178.6, IC181.10
- new net N$534: IC178.8, IC181.12
- new net N$535: IC178.11, IC181.13
- new net N$536: IC179.3, IC182.1
- new net N$537: IC179.6, IC182.2
- new net N$538: IC179.8, IC182.4
- new net N$539: IC179.11, IC182.5
- new net N$540: IC180.3, IC182.9
- new net N$541: IC180.6, IC182.10
- new net N$542: IC180.8, IC182.12
- new net N$543: IC180.11, IC182.13
- new net N$544: IC186.6, IC186.9
- new net N$545: IC186.10, IC186.11
- new net N$546: IC191.6, IC191.9
- new net N$547: IC191.10, IC191.11
- new net N$548: IC191.12, IC191.3, IC191.4
- new net N$549: IC207.6, IC207.9
- new net N$550: IC189.12, IC189.3, IC189.4
- new net N$551: IC189.10, IC189.11
- new net N$552: IC189.6, IC189.9
- new net N$553: IC185.6, IC185.9
- new net N$554: IC185.10, IC185.11
- new net N$555: IC190.12, IC190.3, IC190.4
- new net N$556: IC190.6, IC190.9
- new net N$557: IC190.10, IC190.11
- new net N$558: IC188.10, IC188.11
- new net N$559: IC188.6, IC188.9
- new net N$560: IC188.12, IC188.3, IC188.4
- new net N$561: IC207.10, IC207.11
- new net N$562: IC195.6, IC195.9
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Routing:
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Other:
- board size 304.8 x 254 mm -> 285.6 x 254 mm
- board text added: "22k"
- board text added: "Multiplier"
- board text added: "add description"
- board text added: "add pin descriptions"
- board text added: "gnd"
- board text added: "multiplicand"
- board text added: "multiplier"
- board text added: "product"
- board text added: "vcc"

Commit message: Major updates to schematic. Almost complete except for load/store and non-7004 series.
Parts:
- removed LED1, LED2: (no value), led:LED5MM
- removed R1, R2: 22k, resistor:0207/10
- removed X1, X2: 2534-5, con-3m:PAK100/2500-5-34
- added BENC0, BENC1, BENC10, BENC2, BENC3, BENC4, BENC5, BENC6, BENC7, BENC8, BENC9, IC372, IC373, IC374, IC375, IC376, IC377, IC378, IC379, IC380, IC381, IC383, IC384, IC385, IC386, IC387, IC388, IC389, IC390, IC391, IC392, IC393, IC394, IC395, IC396, IC397, IC398, IC399, IC447, IC448, IC472, IC473, IC474, IC487, IC488, IC489, IC490, IC491, IC492, IC493, IC494, IC495, IC496, IC497, IC498, IC499, IC500, IC501, IC502, IC513, IC514, IC515, IC516, IC517, IC518, IC519, IC520: 74HC00D, 74HC00:SO14
- added IC382, IC400, IC401, IC402, IC403, IC404, IC405, IC406, IC407, IC408, IC409, IC410, IC411, IC412, IC413, IC414, IC415, IC416, IC417, IC418, IC419, IC420, IC421, IC422, IC423, IC424, IC425, IC426, IC427, IC428, IC429, IC430, IC431, IC432, IC433, IC434, IC435, IC436, IC437, IC438, IC439, IC440, IC441, IC442, IC443, IC444, IC445, IC446, IC449, IC450, IC451, IC452, IC453, IC454, IC455, IC456, IC457, IC458, IC459, IC460, IC461, IC462, IC463, IC464, IC465, IC466, IC467, IC468, IC469, IC470, IC471, IC475, IC476, IC477, IC478, IC479, IC480, IC481, IC482, IC483, IC484, IC485, IC486, IC503, IC504, IC505, IC506, IC507, IC508, IC509, IC510, IC511, IC512: 74HC125D, 74HC00:SO14
- IC234, IC235, IC236, IC237, IC238, IC239, IC240, IC241, IC242, IC243, IC244, IC245, IC246, IC247, IC248, IC249, IC293, IC294, IC295, IC296, IC297, IC298, IC299, IC300: value 74HC00D -> 74HC125D
- IC334, IC335, IC336, IC337, IC338, IC339, IC340, IC341, IC342, IC343, IC344, IC345, IC346, IC347, IC348, IC349, IC350, IC351: value 74HC377DW -> 74HC00D; device 74HC00:SO20W -> 74HC00:SO14
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Connections:
- net N$718 renamed SIGN
- net N$905 renamed CMDN6
- net REG14Q2 renamed CMD2
- net REG2Q2 renamed OR_SEL
- removed net AOP: IC242.3, IC244.4, IC247.4, IC251.1, IC254.1, IC256.1, IC265.1, IC267.1, IC270.1
- removed net AREG0: IC243.5
- removed net AREG1: IC249.2, IC263.3
- removed net AREG2: IC253.2, IC263.11
- removed net AREG3: IC253.13
- removed net AREG4: IC258.10
- removed net AREG5: IC259.5
- removed net AREG6: IC269.2
- removed net AREG7: IC269.13
- removed net AWE: IC239.11
- removed net A_MULT0: IC1.1, IC1.2, IC13.10, IC14.5, IC17.13, IC17.2, IC20.10, IC21.5, IC24.13, IC24.2, IC69.2, X1.3
- removed net A_MULT1: IC1.12, IC1.5, IC12.2, IC12.5, IC126.2, IC126.5, IC15.2, IC15.5, IC16.2, IC16.5, IC18.2, IC18.5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
- removed net A_MULT2: IC1.13, IC2.2, IC3.12, IC3.13, X1.7
- removed net A_MULT3: IC154.10, IC154.9, IC157.2, IC157.5, IC26.2, IC26.5, IC29.2, IC29.5, IC3.1, IC3.2, IC30.2, IC30.5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
- removed net A_MULT4: IC5.2, IC5.5, IC7.12, IC7.13, X1.11
- removed net A_MULT5: IC10.4, IC10.5, IC114.2, IC114.5, IC40.2, IC40.5, IC43.2, IC43.5, IC44.2, IC44.5, IC46.2, IC46.5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
- removed net A_MULT6: IC10.1, IC10.2, IC8.5, IC9.2, X1.15
- removed net A_MULT7: IC108.2, IC108.5, IC11.5, IC54.2, IC54.5, IC57.2, IC57.5, IC58.2, IC58.5, IC60.2, IC60.5, IC61.2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
- removed net A_VOP0: IC171.1, IC175.1, IC175.2, IC177.1, IC177.2, IC183.1, IC183.13, IC195.2, IC195.5, IC198.4, IC198.5, IC263.10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
- removed net A_VOP1: IC171.9, IC175.4, IC175.5, IC177.10, IC177.9, IC184.1, IC184.13, IC196.2, IC196.5, IC198.12, IC198.13, X2.5
- removed net A_VOP2: IC172.1, IC175.10, IC175.9, IC178.1, IC178.2, IC185.1, IC185.13, IC197.2, IC197.5, IC200.10, IC200.9, X2.7
- removed net A_VOP3: IC172.9, IC175.12, IC175.13, IC178.10, IC178.9, IC186.1, IC186.13, IC203.4, IC203.5, IC205.2, IC205.5, X2.9
- removed net A_VOP4: IC173.1, IC176.1, IC176.2, IC179.1, IC179.2, IC187.1, IC187.13, IC210.2, IC210.5, IC213.4, IC213.5, X2.11
- removed net A_VOP5: IC173.9, IC176.4, IC176.5, IC179.10, IC179.9, IC188.1, IC188.13, IC211.2, IC211.5, IC213.12, IC213.13, X2.13
- removed net A_VOP6: IC174.1, IC176.10, IC176.9, IC180.1, IC180.2, IC189.1, IC189.13, IC212.2, IC212.5, IC215.10, IC215.9, X2.15
- removed net A_VOP7: IC174.9, IC176.12, IC176.13, IC180.10, IC180.9, IC190.1, IC190.13, IC218.4, IC218.5, IC220.2, IC220.5, X2.17
- removed net BOP: IC242.6, IC244.1, IC247.1, IC251.4, IC254.4, IC256.4, IC265.4, IC267.4, IC270.4
- removed net B_MULT0: IC24.9, IC38.9, IC52.9, IC66.9, IC69.1, IC69.12, IC72.4, IC72.9, X1.19
- removed net B_MULT1: IC21.12, IC24.12, IC35.12, IC38.12, IC49.12, IC52.12, IC63.12, IC66.12, X1.21
- removed net B_MULT2: IC21.1, IC24.1, IC35.1, IC38.1, IC49.1, IC52.1, IC63.1, IC66.1, X1.23
- removed net B_MULT3: IC20.4, IC21.4, IC34.4, IC35.4, IC48.4, IC49.4, IC62.4, IC63.4, X1.25
- removed net B_MULT4: IC17.9, IC20.9, IC31.9, IC34.9, IC45.9, IC48.9, IC59.9, IC62.9, X1.27
- removed net B_MULT5: IC14.12, IC17.12, IC28.12, IC31.12, IC42.12, IC45.12, IC56.12, IC59.12, X1.29
- removed net B_MULT6: IC14.1, IC17.1, IC28.1, IC31.1, IC42.1, IC45.1, IC56.1, IC59.1, X1.31
- removed net B_MULT7: IC13.4, IC13.9, IC14.4, IC27.4, IC27.9, IC28.4, IC41.4, IC41.9, IC42.4, IC55.4, IC55.9, IC56.4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
- removed net B_VOP0: IC171.2, IC177.4, IC177.5, IC183.2, IC183.5, IC191.2, IC191.5, X2.19
- removed net B_VOP1: IC171.10, IC177.12, IC177.13, IC184.2, IC184.5, IC193.2, IC193.5, X2.21
- removed net B_VOP2: IC172.2, IC178.4, IC178.5, IC185.2, IC185.5, IC194.2, IC194.5, X2.23
- removed net B_VOP3: IC172.10, IC178.12, IC178.13, IC186.2, IC186.5, IC204.2, IC204.5, X2.25
- removed net B_VOP4: IC173.2, IC179.4, IC179.5, IC187.2, IC187.5, IC207.2, IC207.5, X2.27
- removed net B_VOP5: IC173.10, IC179.12, IC179.13, IC188.2, IC188.5, IC208.2, IC208.5, X2.29
- removed net B_VOP6: IC174.2, IC180.4, IC180.5, IC189.2, IC189.5, IC209.2, IC209.5, X2.31
- removed net B_VOP7: IC174.10, IC180.12, IC180.13, IC190.2, IC190.5, IC219.2, IC219.5, X2.33
- removed net CCLEAR: X2.22
- removed net CLK: X2.20
- removed net CLK3: IC334.11, IC335.11
- removed net COP: IC242.8, IC245.1, IC248.1, IC252.1, IC255.1, IC257.1, IC266.1, IC268.1, IC271.1
- removed net DOP: IC242.11, IC245.4, IC248.4, IC252.4, IC255.4, IC257.4, IC266.4, IC268.4, IC271.4
- removed net EOP: IC243.3, IC246.1, IC250.12, IC260.12, IC261.12, IC262.12, IC272.12, IC273.12, IC274.12
- removed net FOP: IC239.8, IC243.4, IC249.1, IC253.1, IC253.12, IC258.9, IC259.4, IC269.1, IC269.12
- removed net GND1: IC171.7, IC172.7, IC173.7, IC174.7, IC175.7, IC176.7, IC177.7, IC178.7, IC179.7, IC180.7, IC181.7, IC182.7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
- removed net GND3: IC275.7, IC276.7, IC277.7, IC278.7, IC279.7, IC280.7, IC281.7, IC282.7, IC283.7, IC284.7, IC285.7, IC286.7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
- removed net INST4: IC360.1, IC361.1, IC363.1, IC364.1, IC365.1, IC366.1, IC367.1, IC370.12, IC370.13
- removed net INST4N: IC352.1, IC353.1, IC354.1, IC355.1, IC356.1, IC357.1, IC358.1, IC359.1, IC370.11
- removed net INST5: IC354.9, IC355.9, IC356.2, IC357.2, IC358.2, IC358.9, IC359.2, IC359.9, IC363.9, IC364.2, IC365.2, IC366.2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
- removed net INST5N: IC352.2, IC352.9, IC353.2, IC353.9, IC354.2, IC355.2, IC356.9, IC357.9, IC360.2, IC360.9, IC361.2, IC361.9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
- removed net INST6: IC371.4, IC371.5
- removed net INST6N: IC371.6
- removed net INST7: IC353.10, IC355.10, IC357.10, IC359.10, IC361.10, IC363.10, IC365.10, IC367.10, IC371.1, IC371.2
- removed net INST7N: IC352.10, IC354.10, IC356.10, IC358.10, IC360.10, IC364.10, IC366.10, IC371.3
- removed net MPROD10: IC346.7
- removed net MPROD11: IC346.8
- removed net MPROD12: IC346.13
- removed net MPROD13: IC346.14
- removed net MPROD14: IC346.17
- removed net MPROD15: IC346.18
- removed net MPROD8: IC346.3
- removed net MPROD9: IC346.4
- removed net N$1035 (its old number): IC298.6, IC298.9
- removed net N$1036 (its old number): IC298.10, IC298.11
- removed net N$1037 (its old number): IC298.12, IC298.3, IC298.4
- removed net N$1054 (its old number): IC299.10, IC299.11
- removed net N$1055 (its old number): IC299.8, IC302.1, IC302.13
- removed net N$1056 (its old number): IC302.12, IC302.3, IC302.4
- removed net N$1057 (its old number): IC302.6, IC302.9
- removed net N$1058 (its old number): IC302.10, IC302.11
- removed net N$1059 (its old number): IC295.3, IC295.9
- removed net N$1060 (its old number): IC295.10, IC295.6
- removed net N$1061 (its old number): IC301.3, IC301.5
- removed net N$1064 (its old number): IC296.1, IC301.8
- removed net N$1065 (its old number): IC296.13, IC296.8
- removed net N$1066 (its old number): IC296.12, IC296.6
- removed net N$1126: IC317.11, IC323.4
- removed net N$1127: IC318.2, IC323.11
- removed net N$1128: IC318.1, IC323.8
- removed net N$1132: IC326.6, IC326.9
- removed net N$1133: IC326.11, IC328.1
- removed net N$1134: IC328.6, IC328.9
- removed net N$1135: IC327.1, IC328.11
- removed net N$1136: IC327.6, IC327.9
- removed net N$1137: IC327.11, IC329.1
- removed net N$1138: IC329.6, IC329.9
- removed net N$1139: IC329.11, IC330.2
- removed net N$1140: IC330.6, IC330.9
- removed net N$689 (its old number): IC276.11, IC277.4
- removed net N$700 (its old number): IC229.3, IC229.9
- removed net N$702 (its old number): IC228.3, IC228.9
- removed net N$715 (its old number): IC227.11, IC230.2
- removed net N$721 (its old number): IC244.10, IC244.3
- removed net N$772 (its old number): IC252.10, IC252.6
- removed net N$773 (its old number): IC252.11, IC260.2
- removed net N$780 (its old number): IC254.12, IC254.13, IC254.8
- removed net N$803 (its old number): IC266.3, IC266.9
- removed net N$841 (its old number): IC258.6, IC261.10
- removed net N$856 (its old number): IC263.13, IC263.8
- removed net N$906 (its old number): IC356.12, IC356.13, IC356.8
- removed net N$999 (its old number): IC361.11, IC369.5
- removed net OP0N: IC231.6, IC235.1, IC236.1, IC237.9, IC238.9
- removed net OP1N: IC231.8, IC235.13, IC235.2, IC236.13, IC236.2
- removed net OP2N: IC231.11, IC235.10, IC238.5, IC240.13, IC240.2
- removed net PCG_N0: IC283.12, IC283.3, IC283.4, IC326.1, IC326.2
- removed net PCG_N1: IC288.12, IC288.3, IC288.4, IC326.10
- removed net PCG_N10: IC304.12, IC304.3, IC304.4, IC333.2
- removed net PCG_N11: IC310.12, IC310.3, IC310.4, IC333.10
- removed net PCG_N12: IC316.12, IC316.3, IC316.4, IC332.2
- removed net PCG_N13: IC322.12, IC322.3, IC322.4, IC332.10
- removed net PCG_N14: IC315.12, IC315.3, IC315.4, IC331.2
- removed net PCG_N15: IC321.12, IC321.3, IC321.4
- removed net PCG_N2: IC282.12, IC282.3, IC282.4, IC328.2
- removed net PCG_N3: IC287.12, IC287.3, IC287.4, IC328.10
- removed net PCG_N4: IC294.12, IC294.3, IC294.4, IC327.2
- removed net PCG_N5: IC300.12, IC300.3, IC300.4, IC327.10
- removed net PCG_N6: IC293.12, IC293.3, IC293.4, IC329.2
- removed net PCG_N7: IC299.12, IC299.3, IC299.4, IC329.10
- removed net PCG_N8: IC305.12, IC305.3, IC305.4, IC330.1
- removed net PCG_N9: IC311.12, IC311.3, IC311.4, IC330.10
- removed net PCQ0: IC283.1, IC283.13, IC284.1, IC284.2, IC334.2
- removed net PCQ1: IC284.12, IC284.13, IC288.1, IC288.13, IC334.5
- removed net PCQ10: IC304.1, IC304.13, IC312.10, IC312.9, IC335.6
- removed net PCQ11: IC307.4, IC307.5, IC310.1, IC310.13, IC335.9
- removed net PCQ12: IC316.1, IC316.13, IC317.1, IC317.2, IC335.12
- removed net PCQ13: IC317.12, IC317.13, IC322.1, IC322.13, IC335.15
- removed net PCQ14: IC315.1, IC315.13, IC323.10, IC323.9, IC335.16
- removed net PCQ15: IC321.1, IC321.13, IC335.19
- removed net PCQ2: IC282.1, IC282.13, IC289.10, IC289.9, IC334.6
- removed net PCQ3: IC285.4, IC285.5, IC287.1, IC287.13, IC334.9
- removed net PCQ4: IC294.1, IC294.13, IC295.1, IC295.2, IC334.12
- removed net PCQ5: IC295.12, IC295.13, IC300.1, IC300.13, IC334.15
- removed net PCQ6: IC293.1, IC293.13, IC301.10, IC301.9, IC334.16
- removed net PCQ7: IC296.4, IC296.5, IC299.1, IC299.13, IC334.19
- removed net PCQ8: IC305.1, IC305.13, IC306.1, IC306.2, IC335.2
- removed net PCQ9: IC306.12, IC306.13, IC311.1, IC311.13, IC335.5
- removed net REG01: IC264.9
- removed net REG02: IC263.4
- removed net REG0Q0: IC336.2
- removed net REG0Q1: IC336.5
- removed net REG0Q2: IC336.6
- removed net REG0Q3: IC336.9
- removed net REG0Q4: IC336.12
- removed net REG0Q5: IC336.15
- removed net REG0Q6: IC336.16
- removed net REG0Q7: IC336.19
- removed net REG10Q0: IC346.2
- removed net REG10Q1: IC346.5
- removed net REG10Q2: IC346.6
- removed net REG10Q3: IC346.9
- removed net REG10Q4: IC346.12
- removed net REG10Q5: IC346.15
- removed net REG10Q6: IC346.16
- removed net REG10Q7: IC346.19
- removed net REG11: IC264.12
- removed net REG11Q0: IC347.2
- removed net REG11Q1: IC347.5
- removed net REG11Q2: IC347.6
- removed net REG11Q3: IC347.9
- removed net REG11Q4: IC347.12
- removed net REG11Q5: IC347.15
- removed net REG11Q6: IC347.16
- removed net REG11Q7: IC347.19
- removed net REG12: IC263.9
- removed net REG12Q0: IC348.2
- removed net REG12Q1: IC348.5
- removed net REG12Q2: IC348.6
- removed net REG12Q3: IC348.9
- removed net REG12Q4: IC348.12
- removed net REG12Q5: IC348.15
- removed net REG12Q6: IC348.16
- removed net REG12Q7: IC348.19
- removed net REG13Q0: IC349.2
- removed net REG13Q1: IC349.5
- removed net REG13Q2: IC349.6
- removed net REG13Q3: IC349.9
- removed net REG13Q4: IC349.12
- removed net REG13Q5: IC349.15
- removed net REG13Q6: IC349.16
- removed net REG13Q7: IC349.19
- removed net REG14Q0: IC350.2
- removed net REG14Q1: IC350.5
- removed net REG14Q3: IC350.9
- removed net REG14Q4: IC350.12
- removed net REG14Q5: IC350.15
- removed net REG14Q6: IC350.16
- removed net REG14Q7: IC350.19
- removed net REG15Q0: IC351.2
- removed net REG15Q1: IC351.5
- removed net REG15Q2: IC351.6
- removed net REG15Q3: IC351.9
- removed net REG15Q4: IC351.12
- removed net REG15Q5: IC351.15
- removed net REG15Q6: IC351.16
- removed net REG15Q7: IC351.19
- removed net REG1Q0: IC337.2
- removed net REG1Q1: IC337.5
- removed net REG1Q2: IC337.6
- removed net REG1Q3: IC337.9
- removed net REG1Q4: IC337.12
- removed net REG1Q5: IC337.15
- removed net REG1Q6: IC337.16
- removed net REG1Q7: IC337.19
- removed net REG2Q0: IC338.2
- removed net REG2Q1: IC338.5
- removed net REG2Q3: IC338.9
- removed net REG2Q4: IC338.12
- removed net REG2Q5: IC338.15
- removed net REG2Q6: IC338.16
- removed net REG2Q7: IC338.19
- removed net REG3Q0: IC339.2
- removed net REG3Q1: IC339.5
- removed net REG3Q2: IC339.6
- removed net REG3Q3: IC339.9
- removed net REG3Q4: IC339.12
- removed net REG3Q5: IC339.15
- removed net REG3Q6: IC339.16
- removed net REG3Q7: IC339.19
- removed net REG4Q0: IC340.2
- removed net REG4Q1: IC340.5
- removed net REG4Q2: IC340.6
- removed net REG4Q3: IC340.9
- removed net REG4Q4: IC340.12
- removed net REG4Q5: IC340.15
- removed net REG4Q6: IC340.16
- removed net REG4Q7: IC340.19
- removed net REG5Q0: IC341.2
- removed net REG5Q1: IC341.5
- removed net REG5Q2: IC341.6
- removed net REG5Q3: IC341.9
- removed net REG5Q4: IC341.12
- removed net REG5Q5: IC341.15
- removed net REG5Q6: IC341.16
- removed net REG5Q7: IC341.19
- removed net REG6Q0: IC342.2
- removed net REG6Q1: IC342.5
- removed net REG6Q2: IC342.6
- removed net REG6Q3: IC342.9
- removed net REG6Q4: IC342.12
- removed net REG6Q5: IC342.15
- removed net REG6Q6: IC342.16
- removed net REG6Q7: IC342.19
- removed net REG7Q0: IC343.2
- removed net REG7Q1: IC343.5
- removed net REG7Q2: IC343.6
- removed net REG7Q3: IC343.9
- removed net REG7Q4: IC343.12
- removed net REG7Q5: IC343.15
- removed net REG7Q6: IC343.16
- removed net REG7Q7: IC343.19
- removed net REG8Q0: IC344.2
- removed net REG8Q1: IC344.5
- removed net REG8Q2: IC344.6
- removed net REG8Q3: IC344.9
- removed net REG8Q4: IC344.12
- removed net REG8Q5: IC344.15
- removed net REG8Q6: IC344.16
- removed net REG8Q7: IC344.19
- removed net REG9Q0: IC345.2
- removed net REG9Q1: IC345.5
- removed net REG9Q2: IC345.6
- removed net REG9Q3: IC345.9
- removed net REG9Q4: IC345.12
- removed net REG9Q5: IC345.15
- removed net REG9Q6: IC345.16
- removed net REG9Q7: IC345.19
- removed net REGD0: IC336.3, IC337.3, IC338.3, IC339.3, IC340.3, IC341.3, IC342.3, IC343.3, IC344.3, IC345.3, IC347.3, IC348.3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
- removed net REGD1: IC336.4, IC337.4, IC338.4, IC339.4, IC340.4, IC341.4, IC342.4, IC343.4, IC344.4, IC345.4, IC347.4, IC348.4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
- removed net REGD2: IC336.7, IC337.7, IC338.7, IC339.7, IC340.7, IC341.7, IC342.7, IC343.7, IC344.7, IC345.7, IC347.7, IC348.7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
- removed net REGD3: IC336.8, IC337.8, IC338.8, IC339.8, IC340.8, IC341.8, IC342.8, IC343.8, IC344.8, IC345.8, IC347.8, IC348.8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
- removed net REGD4: IC336.13, IC337.13, IC338.13, IC339.13, IC340.13, IC341.13, IC342.13, IC343.13, IC344.13, IC345.13, IC347.13, IC348.13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
- removed net REGD5: IC336.14, IC337.14, IC338.14, IC339.14, IC340.14, IC341.14, IC342.14, IC343.14, IC344.14, IC345.14, IC347.14, IC348.14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
- removed net REGD6: IC336.17, IC337.17, IC338.17, IC339.17, IC340.17, IC341.17, IC342.17, IC343.17, IC344.17, IC345.17, IC347.17, IC348.17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
- removed net REGD7: IC336.18, IC337.18, IC338.18, IC339.18, IC340.18, IC341.18, IC342.18, IC343.18, IC344.18, IC345.18, IC347.18, IC348.18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
- removed net RES0: IC246.11, X2.4
- removed net RES1: IC250.8, X2.6
- removed net RES2: IC260.8, X2.8
- removed net RES3: IC261.8, X2.10
- removed net RES4: IC262.8, X2.12
- removed net RES5: IC272.8, X2.14
- removed net RES6: IC273.8, X2.16
- removed net RES7: IC274.8, X2.18
- removed net RSEL0N: IC336.1, IC362.3
- removed net RSEL10N: IC346.1
- removed net RSEL11N: IC347.1, IC369.8
- removed net RSEL12N: IC348.1, IC369.11
- removed net RSEL13N: IC349.1, IC370.3
- removed net RSEL14N: IC350.1, IC370.6
- removed net RSEL15N: IC351.1, IC370.8
- removed net RSEL1N: IC337.1, IC362.6
- removed net RSEL2N: IC338.1, IC362.8
- removed net RSEL3N: IC339.1, IC362.11
- removed net RSEL4N: IC340.1, IC368.3
- removed net RSEL5N: IC341.1, IC368.6
- removed net RSEL6N: IC342.1, IC368.8
- removed net RSEL7N: IC343.1, IC368.11
- removed net RSEL8N: IC344.1, IC369.3
- removed net RSEL9N: IC345.1, IC369.6
- removed net SIGN_REG: X2.26
- removed net SUB_SEL_N: IC239.6, IC243.2
- removed net VCC1: IC171.14, IC172.14, IC173.14, IC174.14, IC175.14, IC176.14, IC177.14, IC178.14, IC179.14, IC180.14, IC181.14, IC182.14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
- removed net VCC3: IC275.14, IC276.14, IC277.14, IC278.14, IC279.14, IC280.14, IC281.14, IC282.14, IC283.14, IC284.14, IC285.14, IC286.14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
- removed net Z_REG: X2.28
- new net A0: BENC0.1, BENC0.2, IC13.10, IC14.5, IC17.13, IC17.2, IC171.1, IC175.1, IC175.2, IC177.1, IC177.2, IC183.1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
- new net A1: BENC0.12, BENC0.5, BENC1.4, BENC2.10, BENC2.9, IC12.2, IC12.5, IC126.2, IC126.5, IC15.2, IC15.5, IC16.2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
- new net A2: BENC0.13, BENC1.2, BENC2.12, BENC2.13, IC172.1, IC175.10, IC175.9, IC178.1, IC178.2, IC185.1, IC185.13, IC197.2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
- new net A3: BENC2.1, BENC2.2, BENC3.10, BENC4.1, BENC4.13, BENC6.1, BENC6.2, IC154.10, IC154.9, IC157.2, IC157.5, IC172.9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
- new net A4: BENC4.2, BENC4.5, BENC5.12, BENC5.13, IC173.1, IC176.1, IC176.2, IC179.1, IC179.2, IC187.1, IC187.13, IC210.2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
- new net A5: BENC5.4, BENC5.5, BENC6.13, BENC7.13, BENC8.1, BENC9.4, BENC9.5, IC114.2, IC114.5, IC173.9, IC176.4, IC176.5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
- new net A6: BENC7.5, BENC8.2, BENC9.1, BENC9.2, IC174.1, IC176.10, IC176.9, IC180.1, IC180.2, IC189.1, IC189.13, IC212.2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
- new net A7: BENC10.5, BENC8.10, BENC8.9, IC108.2, IC108.5, IC174.9, IC176.12, IC176.13, IC180.10, IC180.9, IC190.1, IC190.13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
- new net ADDSUB_SEL: IC341.8, IC448.4, IC448.5
- new net ADDSUB_SEL_N: IC448.6, IC487.2
- new net ADD_SEL: IC487.3, IC487.4, IC487.5
- new net ADD_SEL_N: IC466.4, IC468.4, IC471.4, IC476.4, IC478.4, IC479.4, IC484.4, IC486.4, IC487.6, IC488.2
- new net AND_SEL: IC335.6
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Routing:
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Other:
- board size 285.6 x 254 mm -> 304.5 x 254.2 mm
- board text removed: "22k"
- board text removed: "Multiplier"
- board text removed: "add description"
- board text removed: "add pin descriptions"
- board text removed: "gnd"
- board text removed: "multiplicand"
- board text removed: "multiplier"
- board text removed: "product"
- board text removed: "vcc"
