File: Eagle/main.sch (EAGLE design)
At the start: 170 parts, among them M041C 74HC00D, M085C 74HC00D, M0FA30 74HC00D, M0FA31 74HC00D, M0FA40 74HC00D, M0FA41 74HC00D, M0FA50 74HC00D, M0FA51 74HC00D, M0FA60 74HC00D, M0FA61 74HC00D, M0FA70 74HC00D, M0FA71 74HC00D, M0FA80 74HC00D, M0FA81 74HC00D, M0HA0 74HC00D, M0HA1 74HC00D, M0HA2 74HC00D, M120C 74HC00D, M163C 74HC00D, M197C 74HC00D, M1FA10 74HC00D, M1FA11 74HC00D, M1FA20 74HC00D, M1FA21 74HC00D, M1FA30 74HC00D, M1FA31 74HC00D, M1FA40 74HC00D, M1FA41 74HC00D, M1FA50 74HC00D, M1FA51 74HC00D, M1FA60 74HC00D, M1FA61 74HC00D, M1FA70 74HC00D, M1FA71 74HC00D, M1FA80 74HC00D, M1FA81 74HC00D, M1FA90 74HC00D, M1FA91 74HC00D, M1HA0 74HC00D, M241C 74HC00D, M285C 74HC00D, M2FA00 74HC00D, M2FA01 74HC00D, M2HA1 74HC00D, M2HA2 74HC00D, M2HA3 74HC00D, M2HA4 74HC00D, M2HA5 74HC00D, M2HA6 74HC00D, M2HA7 74HC00D, M2HA8 74HC00D

Commit message: SystemVerilog with assigns
Parts:
- removed BEL7, BENC0, BENC10, BENC1_1, BENC2, BENC3, BENC4, BENC5, BENC6, BENC7, BENC8, BENC9, BSEL0, BSEL1, BSEL10, BSEL11, BSEL12, BSEL13, BSEL14, BSEL15, BSEL16, BSEL17, BSEL18, BSEL19, BSEL2, BSEL20, BSEL24, BSEL25, BSEL26, BSEL27, BSEL3, BSEL31, BSEL32, BSEL33, BSEL34, BSEL38, BSEL39, BSEL4, BSEL40, BSEL41, BSEL45, BSEL46, BSEL47, BSEL5, BSEL58, BSEL6, BSEL62, BSEL63, BSEL64, BSEL65, BSEL66, BSEL67, BSEL68, BSEL69, BSEL70, BSEL71, BSEL8, BSEL9, CLA0, CLA1, CLA110, CLA111, CLA120, CLA121, CLA130, CLA131, CLA140, CLA141, CLA150, CLA151, CLA51, CLA6, CLAP0, CLAP1, CLAP2, CLU0, CLU1, CLU2, CLU3, CLU4, CLU5, CLU6, HA1B0, M041C, M085C, M0FA30, M0FA31, M0FA40, M0FA41, M0FA50, M0FA51, M0FA60, M0FA61, M0FA70, M0FA71, M0FA80, M0FA81, M0HA0, M0HA1, M0HA2, M120C, M197C, M1FA10, M1FA11, M1FA20, M1FA21, M1FA70, M1FA71, M1FA80, M1FA81, M1FA90, M1FA91, M1HA0, M285C, M2FA00, M2FA01, M2HA1, M2HA3, M2HA4, M2HA5, M2HA6, M2HA7, M2HA8: 74HC00D, 74HC00:74HC00D
- added IC1, IC10, IC100, IC101, IC102, IC103, IC104, IC105, IC106, IC107, IC108, IC109, IC11, IC110, IC111, IC112, IC113, IC114, IC115, IC116, IC117, IC12, IC120, IC121, IC122, IC123, IC124, IC125, IC126, IC127, IC128, IC13, IC14, IC145, IC15, IC151, IC152, IC153, IC154, IC155, IC156, IC157, IC158, IC159, IC16, IC160, IC161, IC162, IC163, IC164, IC165, IC166, IC167, IC168, IC169, IC17, IC170, IC171, IC172, IC173, IC174, IC175, IC176, IC177, IC178, IC179, IC18, IC180, IC181, IC182, IC183, IC184, IC185, IC186, IC187, IC188, IC189, IC19, IC190, IC191, IC192, IC193, IC194, IC195, IC196, IC197, IC198, IC199, IC2, IC20, IC200, IC201, IC202, IC203, IC204, IC205, IC206, IC207, IC208, IC209, IC21, IC210, IC211, IC212, IC213, IC214, IC215, IC216, IC217, IC218, IC219, IC22, IC220, IC221, IC222, IC223, IC224, IC225, IC226, IC227, IC228, IC229, IC23, IC230, IC231, IC232, IC233, IC234, IC235, IC236, IC237, IC238, IC239, IC24, IC240, IC241, IC242, IC243, IC244, IC245, IC246, IC247, IC248, IC249, IC25, IC250, IC251, IC252, IC253, IC254, IC255, IC256, IC257, IC258, IC259, IC26, IC260, IC261, IC262, IC263, IC264, IC265, IC266, IC267, IC268, IC269, IC270, IC271, IC272, IC273, IC274, IC275, IC276, IC277, IC278, IC279, IC280, IC281, IC282, IC283, IC284, IC285, IC286, IC287, IC288, IC289, IC29, IC290, IC291, IC292, IC293, IC294, IC295, IC296, IC297, IC298, IC299, IC3, IC30, IC300, IC301, IC302, IC303, IC304, IC305, IC306, IC307, IC308, IC309, IC310, IC311, IC312, IC313, IC314, IC315, IC316, IC317, IC318, IC319, IC32, IC320, IC321, IC322, IC323, IC324, IC325, IC326, IC327, IC328, IC329, IC33, IC330, IC331, IC332, IC333, IC352, IC353, IC354, IC355, IC356, IC357, IC358, IC359, IC36, IC360, IC361, IC362, IC363, IC364, IC365, IC366, IC367, IC368, IC369, IC37, IC370, IC371, IC39, IC4, IC40, IC43, IC44, IC46, IC47, IC5, IC50, IC51, IC53, IC54, IC57, IC58, IC6, IC60, IC61, IC62, IC63, IC64, IC65, IC66, IC67, IC68, IC69, IC7, IC70, IC71, IC72, IC73, IC74, IC75, IC76, IC77, IC78, IC79, IC8, IC80, IC81, IC82, IC83, IC84, IC85, IC86, IC87, IC88, IC89, IC9, IC90: 74HC00D, 74HC00:74HC00D
- added IC334, IC335, IC336, IC337, IC338, IC339, IC340, IC341, IC342, IC343, IC344, IC345, IC346, IC347, IC348, IC349, IC350, IC351: 74HC377DW, 74HC00:74HC377DW
- added LED1, LED2: (no value), led:LED5MM
- added R1, R2: 22k, resistor:R-US_0207/10
- added X1, X2: 2534-5, con-3m:2534-5
- renumbered BSEL21 to IC27, BSEL22 to IC28, BSEL23 to IC31, BSEL28 to IC34, BSEL29 to IC35, BSEL30 to IC38, BSEL35 to IC41, BSEL36 to IC42, BSEL37 to IC45, BSEL42 to IC48, BSEL43 to IC49, BSEL44 to IC52, BSEL59 to IC55, BSEL60 to IC56, BSEL61 to IC59, CLA100 to IC130, CLA101 to IC134, CLA20 to IC146, CLA21 to IC149, CLA30 to IC140, CLA31 to IC144, CLA40 to IC147, CLA41 to IC150, CLA50 to IC141, CLA70 to IC135, CLA71 to IC138, CLA80 to IC129, CLA81 to IC133, CLA90 to IC136, CLA91 to IC139, CLAP3 to IC131, CLAP4 to IC137, CLAP5 to IC132, CLAP6 to IC142, CLAP7 to IC148, CLAP8 to IC143, M163C to IC95, M1FA30 to IC97, M1FA31 to IC99, M1FA40 to IC96, M1FA41 to IC98, M1FA50 to IC92, M1FA51 to IC94, M1FA60 to IC91, M1FA61 to IC93, M241C to IC118, M2HA2 to IC119
Connections:
- removed net A0: BEL7C.I1, BENC0A.I0, BENC0A.I1, BSEL0C.I1, BSEL1B.I1, BSEL2A.I1, BSEL2D.I1, BSEL66B.I1, BSEL8B.I1, BSEL9A.I1, BSEL9D.I1
- removed net A1: BENC0B.I1, BENC0D.I0, BENC1_1A.I0, BENC2C.I0, BENC2C.I1, BSEL10B.I1, BSEL10D.I1, BSEL11B.I1, BSEL11D.I1, BSEL12A.I1, BSEL12D.I1, BSEL13A.I1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
- removed net A2: BENC0D.I1, BENC1_1B.I1, BENC2D.I0, BENC2D.I1
- removed net A3: BENC2A.I0, BENC2A.I1, BENC3C.I1, BENC4A.I0, BENC4B.I0, BENC6A.I0, BENC6A.I1, BSEL17B.I1, BSEL17D.I1, BSEL18B.I1, BSEL18D.I1, BSEL19A.I1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
- removed net A4: BENC4A.I1, BENC4C.I1, BENC5D.I0, BENC5D.I1
- removed net A5: BENC5B.I0, BENC5B.I1, BENC6D.I1, BENC7B.I0, BENC7C.I0, BENC9B.I0, BENC9B.I1, BSEL31B.I1, BSEL31D.I1, BSEL32B.I1, BSEL32D.I1, BSEL33A.I1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
- removed net A6: BENC7C.I1, BENC8A.I1, BENC9A.I0, BENC9A.I1
- removed net A7: BENC10B.I1, BENC8C.I0, BENC8C.I1, BSEL45B.I1, BSEL45D.I1, BSEL46B.I1, BSEL46D.I1, BSEL47A.I1, BSEL47D.I1, BSEL58A.I1, BSEL58D.I1, BSEL62B.I1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
- removed net B0: BSEL66B.I0, BSEL66C.I0, BSEL67B.I0, BSEL67C.I0, BSEL9C.I0, IC31C.I0, IC45C.I0, IC59C.I0
- removed net B1: BSEL8D.I0, BSEL9D.I0, IC28D.I0, IC31D.I0, IC42D.I0, IC45D.I0, IC56D.I0, IC59D.I0
- removed net B2: BSEL8A.I0, BSEL9A.I0, IC28A.I0, IC31A.I0, IC42A.I0, IC45A.I0, IC56A.I0, IC59A.I0
- removed net B3: BEL7B.I0, BSEL8B.I0, IC27B.I0, IC28B.I0, IC41B.I0, IC42B.I0, IC55B.I0, IC56B.I0
- removed net B4: BEL7C.I0, BSEL16C.I0, BSEL2C.I0, IC27C.I0, IC38C.I0, IC41C.I0, IC52C.I0, IC55C.I0
- removed net B5: BSEL15D.I0, BSEL16D.I0, BSEL1D.I0, BSEL2D.I0, IC35D.I0, IC38D.I0, IC49D.I0, IC52D.I0
- removed net B6: BSEL15A.I0, BSEL16A.I0, BSEL1A.I0, BSEL2A.I0, IC35A.I0, IC38A.I0, IC49A.I0, IC52A.I0
- removed net B7: BSEL0B.I0, BSEL0C.I0, BSEL14B.I0, BSEL14C.I0, BSEL15B.I0, BSEL1B.I0, IC34B.I0, IC34C.I0, IC35B.I0, IC48B.I0, IC48C.I0, IC49B.I0
- removed net N$444 (its old number): CLAP0A.O, CLAP0C.I0
- removed net N$453 (its old number): CLAP0B.O, CLAP0C.I1
- removed net N$457 (its old number): CLAP1A.O, CLAP1B.I1
- removed net N$458 (its old number): CLAP0D.O, CLAP1B.I0
- removed net N$46 (its old number): BSEL14D.I1, BSEL15A.O
- removed net N$461 (its old number): CLAP1D.O, CLAP2A.I1
- removed net N$462 (its old number): CLAP1C.O, CLAP2A.I0
- removed net N$467 (its old number): CLAP2C.O, CLAP2D.I1
- removed net N$468 (its old number): CLAP2B.O, CLAP2D.I0
- removed net N$51 (its old number): BSEL14D.I0, BSEL15B.O
- removed net N$52 (its old number): BSEL14A.I0, BSEL14C.O
- removed net N$53 (its old number): BSEL14A.I1, BSEL14B.O
- removed net N$54 (its old number): BSEL15C.I1, BSEL15D.O
- removed net N$55 (its old number): BSEL15C.I0, BSEL16A.O
- removed net N$56 (its old number): BSEL16B.I1, BSEL16C.O
- removed net N$57 (its old number): BSEL16B.I0, BSEL16D.O
- removed net PP2_SE_N: HA1B0A.O
- removed net Z10: M2HA8B.I1, M2HA8C.I1
- new net ADD_C0: IC192D.O, IC199A.I1, IC199B.I1, IC222A.I0
- new net ADD_G_N0: IC195A.O, IC195B.I0, IC195D.I0, IC222B.I1
- new net ADD_G_N1: IC196A.O, IC196B.I0, IC196D.I0, IC222D.I1
- new net ADD_G_N2: IC197A.O, IC197B.I0, IC197D.I0, IC223B.I1
- new net ADD_G_N3: IC205A.O, IC205B.I0, IC205D.I0, IC223D.I1
- new net ADD_G_N4: IC210A.O, IC210B.I0, IC210D.I0, IC224B.I1
- new net ADD_G_N5: IC211A.O, IC211B.I0, IC211D.I0, IC224D.I1
- new net ADD_G_N6: IC212A.O, IC212B.I0, IC212D.I0, IC225B.I1
- new net ADD_G_N7: IC220A.O, IC220B.I0, IC220D.I0, IC225D.I1
- new net ADD_P0: IC198C.O, IC222A.I1
- new net ADD_P1: IC200B.O, IC222C.I1
- new net ADD_P2: IC203A.O, IC223A.I1
- new net ADD_P3: IC203D.O, IC223C.I1
- new net ADD_P4: IC213C.O, IC224A.I1
- new net ADD_P5: IC215B.O, IC224C.I1
- new net ADD_P6: IC218A.O, IC225A.I1
- new net ADD_P7: IC218D.O, IC225C.I1
- new net AND0: IC171B.O, IC244B.I1
- new net AND1: IC171D.O, IC247B.I1
- new net AND2: IC172B.O, IC251A.I1
- new net AND3: IC172D.O, IC254A.I1
- new net AND4: IC173B.O, IC256A.I1
- new net AND5: IC173D.O, IC265A.I1
- new net AND6: IC174B.O, IC267A.I1
- new net AND7: IC174D.O, IC270A.I1
- new net AOP: IC242A.O, IC244B.I0, IC247B.I0, IC251A.I0, IC254A.I0, IC256A.I0, IC265A.I0, IC267A.I0, IC270A.I0
- new net AREG0: IC243B.I1
- new net AREG1: IC249A.I1, IC263A.O
- new net AREG2: IC253A.I1, IC263D.O
- new net AREG3: IC253D.I1
- new net AREG4: IC258C.I1
- new net AREG5: IC259B.I1
- new net AREG6: IC269A.I1
- new net AREG7: IC269D.I1
- new net AWE: IC239D.O
- new net A_MULT0: IC13C.I1, IC14B.I1, IC17A.I1, IC17D.I1, IC1A.I0, IC1A.I1, IC20C.I1, IC21B.I1, IC24A.I1, IC24D.I1, IC69A.I1, X1-3.KL
- new net A_MULT1: IC126A.I1, IC126B.I1, IC12A.I1, IC12B.I1, IC15A.I1, IC15B.I1, IC16A.I1, IC16B.I1, IC18A.I1, IC18B.I1, IC19A.I1, IC19B.I1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
- new net A_MULT2: IC1D.I1, IC2A.I1, IC3D.I0, IC3D.I1, X1-7.KL
- new net A_MULT3: IC154C.I0, IC154C.I1, IC157A.I1, IC157B.I1, IC26A.I1, IC26B.I1, IC29A.I1, IC29B.I1, IC30A.I1, IC30B.I1, IC32A.I1, IC32B.I1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
- new net A_MULT4: IC5A.I1, IC5B.I1, IC7D.I0, IC7D.I1, X1-11.KL
- new net A_MULT5: IC10B.I0, IC10B.I1, IC114A.I1, IC114B.I1, IC40A.I1, IC40B.I1, IC43A.I1, IC43B.I1, IC44A.I1, IC44B.I1, IC46A.I1, IC46B.I1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
- new net A_MULT6: IC10A.I0, IC10A.I1, IC8B.I1, IC9A.I1, X1-15.KL
- new net A_MULT7: IC108A.I1, IC108B.I1, IC11B.I1, IC54A.I1, IC54B.I1, IC57A.I1, IC57B.I1, IC58A.I1, IC58B.I1, IC60A.I1, IC60B.I1, IC61A.I1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
- new net A_VOP0: IC171A.I0, IC175A.I0, IC175A.I1, IC177A.I0, IC177A.I1, IC183A.I0, IC183D.I1, IC195A.I1, IC195B.I1, IC198B.I0, IC198B.I1, IC263C.I1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
- new net A_VOP1: IC171C.I0, IC175B.I0, IC175B.I1, IC177C.I0, IC177C.I1, IC184A.I0, IC184D.I1, IC196A.I1, IC196B.I1, IC198D.I0, IC198D.I1, X2-5.KL
- new net A_VOP2: IC172A.I0, IC175C.I0, IC175C.I1, IC178A.I0, IC178A.I1, IC185A.I0, IC185D.I1, IC197A.I1, IC197B.I1, IC200C.I0, IC200C.I1, X2-7.KL
- new net A_VOP3: IC172C.I0, IC175D.I0, IC175D.I1, IC178C.I0, IC178C.I1, IC186A.I0, IC186D.I1, IC203B.I0, IC203B.I1, IC205A.I1, IC205B.I1, X2-9.KL
- new net A_VOP4: IC173A.I0, IC176A.I0, IC176A.I1, IC179A.I0, IC179A.I1, IC187A.I0, IC187D.I1, IC210A.I1, IC210B.I1, IC213B.I0, IC213B.I1, X2-11.KL
- new net A_VOP5: IC173C.I0, IC176B.I0, IC176B.I1, IC179C.I0, IC179C.I1, IC188A.I0, IC188D.I1, IC211A.I1, IC211B.I1, IC213D.I0, IC213D.I1, X2-13.KL
- new net A_VOP6: IC174A.I0, IC176C.I0, IC176C.I1, IC180A.I0, IC180A.I1, IC189A.I0, IC189D.I1, IC212A.I1, IC212B.I1, IC215C.I0, IC215C.I1, X2-15.KL
- new net A_VOP7: IC174C.I0, IC176D.I0, IC176D.I1, IC180C.I0, IC180C.I1, IC190A.I0, IC190D.I1, IC218B.I0, IC218B.I1, IC220A.I1, IC220B.I1, X2-17.KL
- new net BOP: IC242B.O, IC244A.I0, IC247A.I0, IC251B.I0, IC254B.I0, IC256B.I0, IC265B.I0, IC267B.I0, IC270B.I0
- new net B_MULT0: IC24C.I0, IC38C.I0, IC52C.I0, IC66C.I0, IC69A.I0, IC69D.I0, IC72B.I0, IC72C.I0, X1-19.KL
- new net B_MULT1: IC21D.I0, IC24D.I0, IC35D.I0, IC38D.I0, IC49D.I0, IC52D.I0, IC63D.I0, IC66D.I0, X1-21.KL
- new net B_MULT2: IC21A.I0, IC24A.I0, IC35A.I0, IC38A.I0, IC49A.I0, IC52A.I0, IC63A.I0, IC66A.I0, X1-23.KL
- new net B_MULT3: IC20B.I0, IC21B.I0, IC34B.I0, IC35B.I0, IC48B.I0, IC49B.I0, IC62B.I0, IC63B.I0, X1-25.KL
- new net B_MULT4: IC17C.I0, IC20C.I0, IC31C.I0, IC34C.I0, IC45C.I0, IC48C.I0, IC59C.I0, IC62C.I0, X1-27.KL
- new net B_MULT5: IC14D.I0, IC17D.I0, IC28D.I0, IC31D.I0, IC42D.I0, IC45D.I0, IC56D.I0, IC59D.I0, X1-29.KL
- new net B_MULT6: IC14A.I0, IC17A.I0, IC28A.I0, IC31A.I0, IC42A.I0, IC45A.I0, IC56A.I0, IC59A.I0, X1-31.KL
- new net B_MULT7: IC13B.I0, IC13C.I0, IC14B.I0, IC27B.I0, IC27C.I0, IC28B.I0, IC41B.I0, IC41C.I0, IC42B.I0, IC55B.I0, IC55C.I0, IC56B.I0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
- new net B_VOP0: IC171A.I1, IC177B.I0, IC177B.I1, IC183A.I1, IC183B.I1, IC191A.I1, IC191B.I1, X2-19.KL
- new net B_VOP1: IC171C.I1, IC177D.I0, IC177D.I1, IC184A.I1, IC184B.I1, IC193A.I1, IC193B.I1, X2-21.KL
- new net B_VOP2: IC172A.I1, IC178B.I0, IC178B.I1, IC185A.I1, IC185B.I1, IC194A.I1, IC194B.I1, X2-23.KL
- new net B_VOP3: IC172C.I1, IC178D.I0, IC178D.I1, IC186A.I1, IC186B.I1, IC204A.I1, IC204B.I1, X2-25.KL
- new net B_VOP4: IC173A.I1, IC179B.I0, IC179B.I1, IC187A.I1, IC187B.I1, IC207A.I1, IC207B.I1, X2-27.KL
- new net B_VOP5: IC173C.I1, IC179D.I0, IC179D.I1, IC188A.I1, IC188B.I1, IC208A.I1, IC208B.I1, X2-29.KL
- new net B_VOP6: IC174A.I1, IC180B.I0, IC180B.I1, IC189A.I1, IC189B.I1, IC209A.I1, IC209B.I1, X2-31.KL
- new net B_VOP7: IC174C.I1, IC180D.I0, IC180D.I1, IC190A.I1, IC190B.I1, IC219A.I1, IC219B.I1, X2-33.KL
- new net CCLEAR: X2-22.KL
- new net CIN: IC192C.I0
- new net CIN1: IC201A.I1, IC201B.I1, IC222B.O, IC222C.I0
- new net CIN2: IC202A.I1, IC202B.I1, IC222D.O, IC223A.I0
- new net CIN3: IC206A.I1, IC206B.I1, IC223B.O, IC223C.I0
- new net CIN4: IC214A.I1, IC214B.I1, IC223D.O, IC224A.I0
- new net CIN5: IC216A.I1, IC216B.I1, IC224B.O, IC224C.I0
- new net CIN6: IC217A.I1, IC217B.I1, IC224D.O, IC225A.I0
- new net CIN7: IC221A.I1, IC221B.I1, IC225B.O, IC225C.I0
- new net CLK: X2-20.KL
- new net CLK3: IC334A.CLK, IC335A.CLK
- new net COP: IC242C.O, IC245A.I0, IC248A.I0, IC252A.I0, IC255A.I0, IC257A.I0, IC266A.I0, IC268A.I0, IC271A.I0
- new net COUT: IC225D.O
- new net CSEL: IC192A.I0, IC192A.I1, IC192C.I1, X2-24.KL
- new net DOP: IC242D.O, IC245B.I0, IC248B.I0, IC252B.I0, IC255B.I0, IC257B.I0, IC266B.I0, IC268B.I0, IC271B.I0
- new net EOP: IC243A.O, IC246A.I0, IC250D.I0, IC260D.I0, IC261D.I0, IC262D.I0, IC272D.I0, IC273D.I0, IC274D.I0
- new net FOP: IC239C.O, IC243B.I0, IC249A.I0, IC253A.I0, IC253D.I0, IC258C.I0, IC259B.I0, IC269A.I0, IC269D.I0
- new net GND1: IC171P.GND, IC172P.GND, IC173P.GND, IC174P.GND, IC175P.GND, IC176P.GND, IC177P.GND, IC178P.GND, IC179P.GND, IC180P.GND, IC181P.GND, IC182P.GND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
- new net GND3: IC275P.GND, IC276P.GND, IC277P.GND, IC278P.GND, IC279P.GND, IC280P.GND, IC281P.GND, IC282P.GND, IC283P.GND, IC284P.GND, IC285P.GND, IC286P.GND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
- new net INST4: IC360A.I0, IC361A.I0, IC363A.I0, IC364A.I0, IC365A.I0, IC366A.I0, IC367A.I0, IC370D.I0, IC370D.I1
- new net INST4N: IC352A.I0, IC353A.I0, IC354A.I0, IC355A.I0, IC356A.I0, IC357A.I0, IC358A.I0, IC359A.I0, IC370D.O
- new net INST5: IC354C.I0, IC355C.I0, IC356A.I1, IC357A.I1, IC358A.I1, IC358C.I0, IC359A.I1, IC359C.I0, IC363C.I0, IC364A.I1, IC365A.I1, IC366A.I1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
- new net INST5N: IC352A.I1, IC352C.I0, IC353A.I1, IC353C.I0, IC354A.I1, IC355A.I1, IC356C.I0, IC357C.I0, IC360A.I1, IC360C.I0, IC361A.I1, IC361C.I0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
- new net INST6: IC371B.I0, IC371B.I1
- new net INST6N: IC371B.O
- new net INST7: IC353C.I1, IC355C.I1, IC357C.I1, IC359C.I1, IC361C.I1, IC363C.I1, IC365C.I1, IC367C.I1, IC371A.I0, IC371A.I1
- new net INST7N: IC352C.I1, IC354C.I1, IC356C.I1, IC358C.I1, IC360C.I1, IC364C.I1, IC366C.I1, IC371A.O
- new net MPROD10: IC346A.3D
- new net MPROD11: IC346A.4D
- new net MPROD12: IC346A.5D
- new net MPROD13: IC346A.6D
- new net MPROD14: IC346A.7D
- new net MPROD15: IC346A.8D
- new net MPROD8: IC346A.1D
- new net MPROD9: IC346A.2D
- new net N$1007: IC283B.O, IC283C.I0
- new net N$1008: IC283C.I1, IC283D.O
- new net N$1009: IC288C.I1, IC288D.O
- new net N$1010: IC288B.O, IC288C.I0
- new net N$1011: IC288C.O, IC291A.I0, IC291D.I1
- new net N$1012: IC291A.O, IC291B.I0, IC291D.I0
- new net N$1013: IC291B.O, IC291C.I0
- new net N$1014: IC291C.I1, IC291D.O
- new net N$1015: IC286A.O, IC286B.I0, IC286D.I0
- new net N$1016: IC282C.O, IC286A.I0, IC286D.I1
- new net N$1017: IC286C.I1, IC286D.O
- new net N$1018: IC286B.O, IC286C.I0
- new net N$1019: IC282C.I1, IC282D.O
- new net N$1020: IC282B.O, IC282C.I0
- new net N$1021: IC287B.O, IC287C.I0
- new net N$1022: IC287C.I1, IC287D.O
- new net N$1023: IC287C.O, IC290A.I0, IC290D.I1
- new net N$1024: IC290A.O, IC290B.I0, IC290D.I0
- new net N$1025: IC290B.O, IC290C.I0
- new net N$1026: IC290C.I1, IC290D.O
- new net N$1027: IC284A.O, IC284C.I0
- new net N$1028: IC284B.O, IC284C.I1
- new net N$1029: IC289A.O, IC289B.I1
- new net N$1030: IC284D.O, IC289B.I0
- new net N$1031: IC285A.I1, IC289D.O
- new net N$1032: IC285A.I0, IC289C.O
- new net N$1033: IC285C.O, IC285D.I1
- new net N$1034: IC285B.O, IC285D.I0
- new net N$1035: IC298B.O, IC298C.I0
- new net N$1036: IC298C.I1, IC298D.O
- new net N$1037: IC298A.O, IC298B.I0, IC298D.I0
- new net N$1038: IC294C.O, IC298A.I0, IC298D.I1
- new net N$1039: IC294B.O, IC294C.I0
- new net N$1040: IC294C.I1, IC294D.O
- new net N$1041: IC300C.I1, IC300D.O
- new net N$1042: IC300B.O, IC300C.I0
- new net N$1043: IC300C.O, IC303A.I0, IC303D.I1
- new net N$1044: IC303A.O, IC303B.I0, IC303D.I0
- new net N$1045: IC303B.O, IC303C.I0
- new net N$1046: IC303C.I1, IC303D.O
- new net N$1047: IC297A.O, IC297B.I0, IC297D.I0
- new net N$1048: IC293C.O, IC297A.I0, IC297D.I1
- new net N$1049: IC297C.I1, IC297D.O
- new net N$1050: IC297B.O, IC297C.I0
- new net N$1051: IC293C.I1, IC293D.O
- new net N$1052: IC293B.O, IC293C.I0
- new net N$1053: IC299B.O, IC299C.I0
- new net N$1054: IC299C.I1, IC299D.O
- new net N$1055: IC299C.O, IC302A.I0, IC302D.I1
- new net N$1056: IC302A.O, IC302B.I0, IC302D.I0
- new net N$1057: IC302B.O, IC302C.I0
- new net N$1058: IC302C.I1, IC302D.O
- new net N$1059: IC295A.O, IC295C.I0
- new net N$1060: IC295B.O, IC295C.I1
- new net N$1061: IC301A.O, IC301B.I1
- new net N$1062: IC295D.O, IC301B.I0
- new net N$1063: IC296A.I1, IC301D.O
- new net N$1064: IC296A.I0, IC301C.O
- new net N$1065: IC296C.O, IC296D.I1
- new net N$1066: IC296B.O, IC296D.I0
- new net N$1067: IC309B.O, IC309C.I0
- new net N$1068: IC309C.I1, IC309D.O
- new net N$1069: IC309A.O, IC309B.I0, IC309D.I0
- new net N$1070: IC305C.O, IC309A.I0, IC309D.I1
- new net N$1071: IC305B.O, IC305C.I0
- new net N$1072: IC305C.I1, IC305D.O
- new net N$1073: IC311C.I1, IC311D.O
- new net N$1074: IC311B.O, IC311C.I0
- new net N$1075: IC311C.O, IC314A.I0, IC314D.I1
- new net N$1076: IC314A.O, IC314B.I0, IC314D.I0
- new net N$1077: IC314B.O, IC314C.I0
- new net N$1078: IC314C.I1, IC314D.O
- new net N$1079: IC308A.O, IC308B.I0, IC308D.I0
- new net N$1080: IC304C.O, IC308A.I0, IC308D.I1
- new net N$1081: IC308C.I1, IC308D.O
- new net N$1082: IC308B.O, IC308C.I0
- new net N$1083: IC304C.I1, IC304D.O
- new net N$1084: IC304B.O, IC304C.I0
- new net N$1085: IC310B.O, IC310C.I0
- new net N$1086: IC310C.I1, IC310D.O
- new net N$1087: IC310C.O, IC313A.I0, IC313D.I1
- new net N$1088: IC313A.O, IC313B.I0, IC313D.I0
- new net N$1089: IC313B.O, IC313C.I0
- new net N$1090: IC313C.I1, IC313D.O
- new net N$1091: IC306A.O, IC306C.I0
- new net N$1092: IC306B.O, IC306C.I1
- new net N$1093: IC312A.O, IC312B.I1
- new net N$1094: IC306D.O, IC312B.I0
- new net N$1095: IC307A.I1, IC312D.O
- new net N$1096: IC307A.I0, IC312C.O
- new net N$1097: IC307C.O, IC307D.I1
- new net N$1098: IC307B.O, IC307D.I0
- new net N$1099: IC320B.O, IC320C.I0
- new net N$1100: IC320C.I1, IC320D.O
- new net N$1101: IC320A.O, IC320B.I0, IC320D.I0
- new net N$1102: IC316C.O, IC320A.I0, IC320D.I1
- new net N$1103: IC316B.O, IC316C.I0
- new net N$1104: IC316C.I1, IC316D.O
- new net N$1105: IC322C.I1, IC322D.O
- new net N$1106: IC322B.O, IC322C.I0
- new net N$1107: IC322C.O, IC325A.I0, IC325D.I1
- new net N$1108: IC325A.O, IC325B.I0, IC325D.I0
- new net N$1109: IC325B.O, IC325C.I0
- new net N$1110: IC325C.I1, IC325D.O
- new net N$1111: IC319A.O, IC319B.I0, IC319D.I0
- new net N$1112: IC315C.O, IC319A.I0, IC319D.I1
- new net N$1113: IC319C.I1, IC319D.O
- new net N$1114: IC319B.O, IC319C.I0
- new net N$1115: IC315C.I1, IC315D.O
- new net N$1116: IC315B.O, IC315C.I0
- new net N$1117: IC321B.O, IC321C.I0
- new net N$1118: IC321C.I1, IC321D.O
- new net N$1119: IC321C.O, IC324A.I0, IC324D.I1
- new net N$1120: IC324A.O, IC324B.I0, IC324D.I0
- new net N$1121: IC324B.O, IC324C.I0
- new net N$1122: IC324C.I1, IC324D.O
- new net N$1123: IC317A.O, IC317C.I0
- new net N$1124: IC317B.O, IC317C.I1
- new net N$1125: IC323A.O, IC323B.I1
- new net N$1126: IC317D.O, IC323B.I0
- new net N$1127: IC318A.I1, IC323D.O
- new net N$1128: IC318A.I0, IC323C.O
- new net N$1132: IC326B.O, IC326C.I0
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Other:
- note added: "AND"
- note added: "NOT"
- note added: "OR"
- note added: "PC"
- note added: "XOR"

Commit message: Major updates to schematic. Almost complete except for load/store and non-7004 series.
Parts:
- removed LED1, LED2: (no value), led:LED5MM
- removed R1, R2: 22k, resistor:R-US_0207/10
- removed X1, X2: 2534-5, con-3m:2534-5
- added BENC0, BENC1, BENC10, BENC2, BENC3, BENC4, BENC5, BENC6, BENC7, BENC8, BENC9, IC372, IC373, IC374, IC375, IC376, IC377, IC378, IC379, IC380, IC381, IC383, IC384, IC385, IC386, IC387, IC388, IC389, IC390, IC391, IC392, IC393, IC394, IC395, IC396, IC397, IC398, IC399, IC447, IC448, IC472, IC473, IC474, IC487, IC488, IC489, IC490, IC491, IC492, IC493, IC494, IC495, IC496, IC497, IC498, IC499, IC500, IC501, IC502, IC513, IC514, IC515, IC516, IC517, IC518, IC519, IC520: 74HC00D, 74HC00:74HC00D
- added IC382, IC400, IC401, IC402, IC403, IC404, IC405, IC406, IC407, IC408, IC409, IC410, IC411, IC412, IC413, IC414, IC415, IC416, IC417, IC418, IC419, IC420, IC421, IC422, IC423, IC424, IC425, IC426, IC427, IC428, IC429, IC430, IC431, IC432, IC433, IC434, IC435, IC436, IC437, IC438, IC439, IC440, IC441, IC442, IC443, IC444, IC445, IC446, IC449, IC450, IC451, IC452, IC453, IC454, IC455, IC456, IC457, IC458, IC459, IC460, IC461, IC462, IC463, IC464, IC465, IC466, IC467, IC468, IC469, IC470, IC471, IC475, IC476, IC477, IC478, IC479, IC480, IC481, IC482, IC483, IC484, IC485, IC486, IC503, IC504, IC505, IC506, IC507, IC508, IC509, IC510, IC511, IC512: 74HC125D, 74HC00:74HC125D
- IC234, IC235, IC236, IC237, IC238, IC239, IC240, IC241, IC242, IC243, IC244, IC245, IC246, IC247, IC248, IC249, IC293, IC294, IC295, IC296, IC297, IC298, IC299, IC300: value 74HC00D -> 74HC125D; device 74HC00:74HC00D -> 74HC00:74HC125D
- IC334, IC335, IC336, IC337, IC338, IC339, IC340, IC341, IC342, IC343, IC344, IC345, IC346, IC347, IC348, IC349, IC350, IC351: value 74HC377DW -> 74HC00D; device 74HC00:74HC377DW -> 74HC00:74HC00D
Connections:
- net N$718 renamed SIGN
- net N$905 renamed CMDN6
- removed net AOP: IC242A.O, IC244B.I0, IC247B.I0, IC251A.I0, IC254A.I0, IC256A.I0, IC265A.I0, IC267A.I0, IC270A.I0
- removed net AREG0: IC243B.I1
- removed net AREG1: IC249A.I1, IC263A.O
- removed net AREG2: IC253A.I1, IC263D.O
- removed net AREG3: IC253D.I1
- removed net AREG4: IC258C.I1
- removed net AREG5: IC259B.I1
- removed net AREG6: IC269A.I1
- removed net AREG7: IC269D.I1
- removed net AWE: IC239D.O
- removed net A_MULT0: IC13C.I1, IC14B.I1, IC17A.I1, IC17D.I1, IC1A.I0, IC1A.I1, IC20C.I1, IC21B.I1, IC24A.I1, IC24D.I1, IC69A.I1, X1-3.KL
- removed net A_MULT1: IC126A.I1, IC126B.I1, IC12A.I1, IC12B.I1, IC15A.I1, IC15B.I1, IC16A.I1, IC16B.I1, IC18A.I1, IC18B.I1, IC19A.I1, IC19B.I1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
- removed net A_MULT2: IC1D.I1, IC2A.I1, IC3D.I0, IC3D.I1, X1-7.KL
- removed net A_MULT3: IC154C.I0, IC154C.I1, IC157A.I1, IC157B.I1, IC26A.I1, IC26B.I1, IC29A.I1, IC29B.I1, IC30A.I1, IC30B.I1, IC32A.I1, IC32B.I1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
- removed net A_MULT4: IC5A.I1, IC5B.I1, IC7D.I0, IC7D.I1, X1-11.KL
- removed net A_MULT5: IC10B.I0, IC10B.I1, IC114A.I1, IC114B.I1, IC40A.I1, IC40B.I1, IC43A.I1, IC43B.I1, IC44A.I1, IC44B.I1, IC46A.I1, IC46B.I1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
- removed net A_MULT6: IC10A.I0, IC10A.I1, IC8B.I1, IC9A.I1, X1-15.KL
- removed net A_MULT7: IC108A.I1, IC108B.I1, IC11B.I1, IC54A.I1, IC54B.I1, IC57A.I1, IC57B.I1, IC58A.I1, IC58B.I1, IC60A.I1, IC60B.I1, IC61A.I1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
- removed net A_VOP0: IC171A.I0, IC175A.I0, IC175A.I1, IC177A.I0, IC177A.I1, IC183A.I0, IC183D.I1, IC195A.I1, IC195B.I1, IC198B.I0, IC198B.I1, IC263C.I1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
- removed net A_VOP1: IC171C.I0, IC175B.I0, IC175B.I1, IC177C.I0, IC177C.I1, IC184A.I0, IC184D.I1, IC196A.I1, IC196B.I1, IC198D.I0, IC198D.I1, X2-5.KL
- removed net A_VOP2: IC172A.I0, IC175C.I0, IC175C.I1, IC178A.I0, IC178A.I1, IC185A.I0, IC185D.I1, IC197A.I1, IC197B.I1, IC200C.I0, IC200C.I1, X2-7.KL
- removed net A_VOP3: IC172C.I0, IC175D.I0, IC175D.I1, IC178C.I0, IC178C.I1, IC186A.I0, IC186D.I1, IC203B.I0, IC203B.I1, IC205A.I1, IC205B.I1, X2-9.KL
- removed net A_VOP4: IC173A.I0, IC176A.I0, IC176A.I1, IC179A.I0, IC179A.I1, IC187A.I0, IC187D.I1, IC210A.I1, IC210B.I1, IC213B.I0, IC213B.I1, X2-11.KL
- removed net A_VOP5: IC173C.I0, IC176B.I0, IC176B.I1, IC179C.I0, IC179C.I1, IC188A.I0, IC188D.I1, IC211A.I1, IC211B.I1, IC213D.I0, IC213D.I1, X2-13.KL
- removed net A_VOP6: IC174A.I0, IC176C.I0, IC176C.I1, IC180A.I0, IC180A.I1, IC189A.I0, IC189D.I1, IC212A.I1, IC212B.I1, IC215C.I0, IC215C.I1, X2-15.KL
- removed net A_VOP7: IC174C.I0, IC176D.I0, IC176D.I1, IC180C.I0, IC180C.I1, IC190A.I0, IC190D.I1, IC218B.I0, IC218B.I1, IC220A.I1, IC220B.I1, X2-17.KL
- removed net BOP: IC242B.O, IC244A.I0, IC247A.I0, IC251B.I0, IC254B.I0, IC256B.I0, IC265B.I0, IC267B.I0, IC270B.I0
- removed net B_MULT0: IC24C.I0, IC38C.I0, IC52C.I0, IC66C.I0, IC69A.I0, IC69D.I0, IC72B.I0, IC72C.I0, X1-19.KL
- removed net B_MULT1: IC21D.I0, IC24D.I0, IC35D.I0, IC38D.I0, IC49D.I0, IC52D.I0, IC63D.I0, IC66D.I0, X1-21.KL
- removed net B_MULT2: IC21A.I0, IC24A.I0, IC35A.I0, IC38A.I0, IC49A.I0, IC52A.I0, IC63A.I0, IC66A.I0, X1-23.KL
- removed net B_MULT3: IC20B.I0, IC21B.I0, IC34B.I0, IC35B.I0, IC48B.I0, IC49B.I0, IC62B.I0, IC63B.I0, X1-25.KL
- removed net B_MULT4: IC17C.I0, IC20C.I0, IC31C.I0, IC34C.I0, IC45C.I0, IC48C.I0, IC59C.I0, IC62C.I0, X1-27.KL
- removed net B_MULT5: IC14D.I0, IC17D.I0, IC28D.I0, IC31D.I0, IC42D.I0, IC45D.I0, IC56D.I0, IC59D.I0, X1-29.KL
- removed net B_MULT6: IC14A.I0, IC17A.I0, IC28A.I0, IC31A.I0, IC42A.I0, IC45A.I0, IC56A.I0, IC59A.I0, X1-31.KL
- removed net B_MULT7: IC13B.I0, IC13C.I0, IC14B.I0, IC27B.I0, IC27C.I0, IC28B.I0, IC41B.I0, IC41C.I0, IC42B.I0, IC55B.I0, IC55C.I0, IC56B.I0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
- removed net B_VOP0: IC171A.I1, IC177B.I0, IC177B.I1, IC183A.I1, IC183B.I1, IC191A.I1, IC191B.I1, X2-19.KL
- removed net B_VOP1: IC171C.I1, IC177D.I0, IC177D.I1, IC184A.I1, IC184B.I1, IC193A.I1, IC193B.I1, X2-21.KL
- removed net B_VOP2: IC172A.I1, IC178B.I0, IC178B.I1, IC185A.I1, IC185B.I1, IC194A.I1, IC194B.I1, X2-23.KL
- removed net B_VOP3: IC172C.I1, IC178D.I0, IC178D.I1, IC186A.I1, IC186B.I1, IC204A.I1, IC204B.I1, X2-25.KL
- removed net B_VOP4: IC173A.I1, IC179B.I0, IC179B.I1, IC187A.I1, IC187B.I1, IC207A.I1, IC207B.I1, X2-27.KL
- removed net B_VOP5: IC173C.I1, IC179D.I0, IC179D.I1, IC188A.I1, IC188B.I1, IC208A.I1, IC208B.I1, X2-29.KL
- removed net B_VOP6: IC174A.I1, IC180B.I0, IC180B.I1, IC189A.I1, IC189B.I1, IC209A.I1, IC209B.I1, X2-31.KL
- removed net B_VOP7: IC174C.I1, IC180D.I0, IC180D.I1, IC190A.I1, IC190B.I1, IC219A.I1, IC219B.I1, X2-33.KL
- removed net CCLEAR: X2-22.KL
- removed net CLK: X2-20.KL
- removed net CLK3: IC334A.CLK, IC335A.CLK
- removed net COP: IC242C.O, IC245A.I0, IC248A.I0, IC252A.I0, IC255A.I0, IC257A.I0, IC266A.I0, IC268A.I0, IC271A.I0
- removed net DOP: IC242D.O, IC245B.I0, IC248B.I0, IC252B.I0, IC255B.I0, IC257B.I0, IC266B.I0, IC268B.I0, IC271B.I0
- removed net EOP: IC243A.O, IC246A.I0, IC250D.I0, IC260D.I0, IC261D.I0, IC262D.I0, IC272D.I0, IC273D.I0, IC274D.I0
- removed net FOP: IC239C.O, IC243B.I0, IC249A.I0, IC253A.I0, IC253D.I0, IC258C.I0, IC259B.I0, IC269A.I0, IC269D.I0
- removed net GND1: IC171P.GND, IC172P.GND, IC173P.GND, IC174P.GND, IC175P.GND, IC176P.GND, IC177P.GND, IC178P.GND, IC179P.GND, IC180P.GND, IC181P.GND, IC182P.GND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
- removed net GND3: IC275P.GND, IC276P.GND, IC277P.GND, IC278P.GND, IC279P.GND, IC280P.GND, IC281P.GND, IC282P.GND, IC283P.GND, IC284P.GND, IC285P.GND, IC286P.GND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
- removed net INST4: IC360A.I0, IC361A.I0, IC363A.I0, IC364A.I0, IC365A.I0, IC366A.I0, IC367A.I0, IC370D.I0, IC370D.I1
- removed net INST4N: IC352A.I0, IC353A.I0, IC354A.I0, IC355A.I0, IC356A.I0, IC357A.I0, IC358A.I0, IC359A.I0, IC370D.O
- removed net INST5: IC354C.I0, IC355C.I0, IC356A.I1, IC357A.I1, IC358A.I1, IC358C.I0, IC359A.I1, IC359C.I0, IC363C.I0, IC364A.I1, IC365A.I1, IC366A.I1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
- removed net INST5N: IC352A.I1, IC352C.I0, IC353A.I1, IC353C.I0, IC354A.I1, IC355A.I1, IC356C.I0, IC357C.I0, IC360A.I1, IC360C.I0, IC361A.I1, IC361C.I0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
- removed net INST6: IC371B.I0, IC371B.I1
- removed net INST6N: IC371B.O
- removed net INST7: IC353C.I1, IC355C.I1, IC357C.I1, IC359C.I1, IC361C.I1, IC363C.I1, IC365C.I1, IC367C.I1, IC371A.I0, IC371A.I1
- removed net INST7N: IC352C.I1, IC354C.I1, IC356C.I1, IC358C.I1, IC360C.I1, IC364C.I1, IC366C.I1, IC371A.O
- removed net MPROD10: IC346A.3D
- removed net MPROD11: IC346A.4D
- removed net MPROD12: IC346A.5D
- removed net MPROD13: IC346A.6D
- removed net MPROD14: IC346A.7D
- removed net MPROD15: IC346A.8D
- removed net MPROD8: IC346A.1D
- removed net MPROD9: IC346A.2D
- removed net N$1035 (its old number): IC298B.O, IC298C.I0
- removed net N$1036 (its old number): IC298C.I1, IC298D.O
- removed net N$1037 (its old number): IC298A.O, IC298B.I0, IC298D.I0
- removed net N$1054 (its old number): IC299C.I1, IC299D.O
- removed net N$1055 (its old number): IC299C.O, IC302A.I0, IC302D.I1
- removed net N$1056 (its old number): IC302A.O, IC302B.I0, IC302D.I0
- removed net N$1057 (its old number): IC302B.O, IC302C.I0
- removed net N$1058 (its old number): IC302C.I1, IC302D.O
- removed net N$1059 (its old number): IC295A.O, IC295C.I0
- removed net N$1060 (its old number): IC295B.O, IC295C.I1
- removed net N$1061 (its old number): IC301A.O, IC301B.I1
- removed net N$1064 (its old number): IC296A.I0, IC301C.O
- removed net N$1065 (its old number): IC296C.O, IC296D.I1
- removed net N$1066 (its old number): IC296B.O, IC296D.I0
- removed net N$1126: IC317D.O, IC323B.I0
- removed net N$1127: IC318A.I1, IC323D.O
- removed net N$1128: IC318A.I0, IC323C.O
- removed net N$1132: IC326B.O, IC326C.I0
- removed net N$1133: IC326D.O, IC328A.I0
- removed net N$1134: IC328B.O, IC328C.I0
- removed net N$1135: IC327A.I0, IC328D.O
- removed net N$1136: IC327B.O, IC327C.I0
- removed net N$1137: IC327D.O, IC329A.I0
- removed net N$1138: IC329B.O, IC329C.I0
- removed net N$1139: IC329D.O, IC330A.I1
- removed net N$1140: IC330B.O, IC330C.I0
- removed net N$689 (its old number): IC276D.O, IC277B.I0
- removed net N$700 (its old number): IC229A.O, IC229C.I0
- removed net N$702 (its old number): IC228A.O, IC228C.I0
- removed net N$715 (its old number): IC227D.O, IC230A.I1
- removed net N$721 (its old number): IC244A.O, IC244C.I1
- removed net N$772 (its old number): IC252B.O, IC252C.I1
- removed net N$773 (its old number): IC252D.O, IC260A.I1
- removed net N$780 (its old number): IC254C.O, IC254D.I0, IC254D.I1
- removed net N$803 (its old number): IC266A.O, IC266C.I0
- removed net N$841 (its old number): IC258B.O, IC261C.I1
- removed net N$856 (its old number): IC263C.O, IC263D.I1
- removed net N$906 (its old number): IC356C.O, IC356D.I0, IC356D.I1
- removed net N$999 (its old number): IC361D.O, IC369B.I1
- removed net OP0N: IC231B.O, IC235A.I0, IC236A.I0, IC237C.I0, IC238C.I0
- removed net OP1N: IC231C.O, IC235A.I1, IC235D.I1, IC236A.I1, IC236D.I1
- removed net OP2N: IC231D.O, IC235C.I1, IC238B.I1, IC240A.I1, IC240D.I1
- removed net PCG_N0: IC283A.O, IC283B.I0, IC283D.I0, IC326A.I0, IC326A.I1
- removed net PCG_N1: IC288A.O, IC288B.I0, IC288D.I0, IC326C.I1
- removed net PCG_N10: IC304A.O, IC304B.I0, IC304D.I0, IC333A.I1
- removed net PCG_N11: IC310A.O, IC310B.I0, IC310D.I0, IC333C.I1
- removed net PCG_N12: IC316A.O, IC316B.I0, IC316D.I0, IC332A.I1
- removed net PCG_N13: IC322A.O, IC322B.I0, IC322D.I0, IC332C.I1
- removed net PCG_N14: IC315A.O, IC315B.I0, IC315D.I0, IC331A.I1
- removed net PCG_N15: IC321A.O, IC321B.I0, IC321D.I0
- removed net PCG_N2: IC282A.O, IC282B.I0, IC282D.I0, IC328A.I1
- removed net PCG_N3: IC287A.O, IC287B.I0, IC287D.I0, IC328C.I1
- removed net PCG_N4: IC294A.O, IC294B.I0, IC294D.I0, IC327A.I1
- removed net PCG_N5: IC300A.O, IC300B.I0, IC300D.I0, IC327C.I1
- removed net PCG_N6: IC293A.O, IC293B.I0, IC293D.I0, IC329A.I1
- removed net PCG_N7: IC299A.O, IC299B.I0, IC299D.I0, IC329C.I1
- removed net PCG_N8: IC305A.O, IC305B.I0, IC305D.I0, IC330A.I0
- removed net PCG_N9: IC311A.O, IC311B.I0, IC311D.I0, IC330C.I1
- removed net PCQ0: IC283A.I0, IC283D.I1, IC284A.I0, IC284A.I1, IC334A.1Q
- removed net PCQ1: IC284D.I0, IC284D.I1, IC288A.I0, IC288D.I1, IC334A.2Q
- removed net PCQ10: IC304A.I0, IC304D.I1, IC312C.I0, IC312C.I1, IC335A.3Q
- removed net PCQ11: IC307B.I0, IC307B.I1, IC310A.I0, IC310D.I1, IC335A.4Q
- removed net PCQ12: IC316A.I0, IC316D.I1, IC317A.I0, IC317A.I1, IC335A.5Q
- removed net PCQ13: IC317D.I0, IC317D.I1, IC322A.I0, IC322D.I1, IC335A.6Q
- removed net PCQ14: IC315A.I0, IC315D.I1, IC323C.I0, IC323C.I1, IC335A.7Q
- removed net PCQ15: IC321A.I0, IC321D.I1, IC335A.8Q
- removed net PCQ2: IC282A.I0, IC282D.I1, IC289C.I0, IC289C.I1, IC334A.3Q
- removed net PCQ3: IC285B.I0, IC285B.I1, IC287A.I0, IC287D.I1, IC334A.4Q
- removed net PCQ4: IC294A.I0, IC294D.I1, IC295A.I0, IC295A.I1, IC334A.5Q
- removed net PCQ5: IC295D.I0, IC295D.I1, IC300A.I0, IC300D.I1, IC334A.6Q
- removed net PCQ6: IC293A.I0, IC293D.I1, IC301C.I0, IC301C.I1, IC334A.7Q
- removed net PCQ7: IC296B.I0, IC296B.I1, IC299A.I0, IC299D.I1, IC334A.8Q
- removed net PCQ8: IC305A.I0, IC305D.I1, IC306A.I0, IC306A.I1, IC335A.1Q
- removed net PCQ9: IC306D.I0, IC306D.I1, IC311A.I0, IC311D.I1, IC335A.2Q
- removed net REG01: IC264C.I0
- removed net REG02: IC263B.I0
- removed net REG0Q0: IC336A.1Q
- removed net REG0Q1: IC336A.2Q
- removed net REG0Q2: IC336A.3Q
- removed net REG0Q3: IC336A.4Q
- removed net REG0Q4: IC336A.5Q
- removed net REG0Q5: IC336A.6Q
- removed net REG0Q6: IC336A.7Q
- removed net REG0Q7: IC336A.8Q
- removed net REG10Q0: IC346A.1Q
- removed net REG10Q1: IC346A.2Q
- removed net REG10Q2: IC346A.3Q
- removed net REG10Q3: IC346A.4Q
- removed net REG10Q4: IC346A.5Q
- removed net REG10Q5: IC346A.6Q
- removed net REG10Q6: IC346A.7Q
- removed net REG10Q7: IC346A.8Q
- removed net REG11: IC264D.I0
- removed net REG11Q0: IC347A.1Q
- removed net REG11Q1: IC347A.2Q
- removed net REG11Q2: IC347A.3Q
- removed net REG11Q3: IC347A.4Q
- removed net REG11Q4: IC347A.5Q
- removed net REG11Q5: IC347A.6Q
- removed net REG11Q6: IC347A.7Q
- removed net REG11Q7: IC347A.8Q
- removed net REG12: IC263C.I0
- removed net REG12Q0: IC348A.1Q
- removed net REG12Q1: IC348A.2Q
- removed net REG12Q2: IC348A.3Q
- removed net REG12Q3: IC348A.4Q
- removed net REG12Q4: IC348A.5Q
- removed net REG12Q5: IC348A.6Q
- removed net REG12Q6: IC348A.7Q
- removed net REG12Q7: IC348A.8Q
- removed net REG13Q0: IC349A.1Q
- removed net REG13Q1: IC349A.2Q
- removed net REG13Q2: IC349A.3Q
- removed net REG13Q3: IC349A.4Q
- removed net REG13Q4: IC349A.5Q
- removed net REG13Q5: IC349A.6Q
- removed net REG13Q6: IC349A.7Q
- removed net REG13Q7: IC349A.8Q
- removed net REG14Q0: IC350A.1Q
- removed net REG14Q1: IC350A.2Q
- removed net REG14Q2: IC350A.3Q
- removed net REG14Q3: IC350A.4Q
- removed net REG14Q4: IC350A.5Q
- removed net REG14Q5: IC350A.6Q
- removed net REG14Q6: IC350A.7Q
- removed net REG14Q7: IC350A.8Q
- removed net REG15Q0: IC351A.1Q
- removed net REG15Q1: IC351A.2Q
- removed net REG15Q2: IC351A.3Q
- removed net REG15Q3: IC351A.4Q
- removed net REG15Q4: IC351A.5Q
- removed net REG15Q5: IC351A.6Q
- removed net REG15Q6: IC351A.7Q
- removed net REG15Q7: IC351A.8Q
- removed net REG1Q0: IC337A.1Q
- removed net REG1Q1: IC337A.2Q
- removed net REG1Q2: IC337A.3Q
- removed net REG1Q3: IC337A.4Q
- removed net REG1Q4: IC337A.5Q
- removed net REG1Q5: IC337A.6Q
- removed net REG1Q6: IC337A.7Q
- removed net REG1Q7: IC337A.8Q
- removed net REG2Q0: IC338A.1Q
- removed net REG2Q1: IC338A.2Q
- removed net REG2Q2: IC338A.3Q
- removed net REG2Q3: IC338A.4Q
- removed net REG2Q4: IC338A.5Q
- removed net REG2Q5: IC338A.6Q
- removed net REG2Q6: IC338A.7Q
- removed net REG2Q7: IC338A.8Q
- removed net REG3Q0: IC339A.1Q
- removed net REG3Q1: IC339A.2Q
- removed net REG3Q2: IC339A.3Q
- removed net REG3Q3: IC339A.4Q
- removed net REG3Q4: IC339A.5Q
- removed net REG3Q5: IC339A.6Q
- removed net REG3Q6: IC339A.7Q
- removed net REG3Q7: IC339A.8Q
- removed net REG4Q0: IC340A.1Q
- removed net REG4Q1: IC340A.2Q
- removed net REG4Q2: IC340A.3Q
- removed net REG4Q3: IC340A.4Q
- removed net REG4Q4: IC340A.5Q
- removed net REG4Q5: IC340A.6Q
- removed net REG4Q6: IC340A.7Q
- removed net REG4Q7: IC340A.8Q
- removed net REG5Q0: IC341A.1Q
- removed net REG5Q1: IC341A.2Q
- removed net REG5Q2: IC341A.3Q
- removed net REG5Q3: IC341A.4Q
- removed net REG5Q4: IC341A.5Q
- removed net REG5Q5: IC341A.6Q
- removed net REG5Q6: IC341A.7Q
- removed net REG5Q7: IC341A.8Q
- removed net REG6Q0: IC342A.1Q
- removed net REG6Q1: IC342A.2Q
- removed net REG6Q2: IC342A.3Q
- removed net REG6Q3: IC342A.4Q
- removed net REG6Q4: IC342A.5Q
- removed net REG6Q5: IC342A.6Q
- removed net REG6Q6: IC342A.7Q
- removed net REG6Q7: IC342A.8Q
- removed net REG7Q0: IC343A.1Q
- removed net REG7Q1: IC343A.2Q
- removed net REG7Q2: IC343A.3Q
- removed net REG7Q3: IC343A.4Q
- removed net REG7Q4: IC343A.5Q
- removed net REG7Q5: IC343A.6Q
- removed net REG7Q6: IC343A.7Q
- removed net REG7Q7: IC343A.8Q
- removed net REG8Q0: IC344A.1Q
- removed net REG8Q1: IC344A.2Q
- removed net REG8Q2: IC344A.3Q
- removed net REG8Q3: IC344A.4Q
- removed net REG8Q4: IC344A.5Q
- removed net REG8Q5: IC344A.6Q
- removed net REG8Q6: IC344A.7Q
- removed net REG8Q7: IC344A.8Q
- removed net REG9Q0: IC345A.1Q
- removed net REG9Q1: IC345A.2Q
- removed net REG9Q2: IC345A.3Q
- removed net REG9Q3: IC345A.4Q
- removed net REG9Q4: IC345A.5Q
- removed net REG9Q5: IC345A.6Q
- removed net REG9Q6: IC345A.7Q
- removed net REG9Q7: IC345A.8Q
- removed net REGD0: IC336A.1D, IC337A.1D, IC338A.1D, IC339A.1D, IC340A.1D, IC341A.1D, IC342A.1D, IC343A.1D, IC344A.1D, IC345A.1D, IC347A.1D, IC348A.1D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
- removed net REGD1: IC336A.2D, IC337A.2D, IC338A.2D, IC339A.2D, IC340A.2D, IC341A.2D, IC342A.2D, IC343A.2D, IC344A.2D, IC345A.2D, IC347A.2D, IC348A.2D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
- removed net REGD2: IC336A.3D, IC337A.3D, IC338A.3D, IC339A.3D, IC340A.3D, IC341A.3D, IC342A.3D, IC343A.3D, IC344A.3D, IC345A.3D, IC347A.3D, IC348A.3D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
- removed net REGD3: IC336A.4D, IC337A.4D, IC338A.4D, IC339A.4D, IC340A.4D, IC341A.4D, IC342A.4D, IC343A.4D, IC344A.4D, IC345A.4D, IC347A.4D, IC348A.4D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
- removed net REGD4: IC336A.5D, IC337A.5D, IC338A.5D, IC339A.5D, IC340A.5D, IC341A.5D, IC342A.5D, IC343A.5D, IC344A.5D, IC345A.5D, IC347A.5D, IC348A.5D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
- removed net REGD5: IC336A.6D, IC337A.6D, IC338A.6D, IC339A.6D, IC340A.6D, IC341A.6D, IC342A.6D, IC343A.6D, IC344A.6D, IC345A.6D, IC347A.6D, IC348A.6D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
- removed net REGD6: IC336A.7D, IC337A.7D, IC338A.7D, IC339A.7D, IC340A.7D, IC341A.7D, IC342A.7D, IC343A.7D, IC344A.7D, IC345A.7D, IC347A.7D, IC348A.7D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
- removed net REGD7: IC336A.8D, IC337A.8D, IC338A.8D, IC339A.8D, IC340A.8D, IC341A.8D, IC342A.8D, IC343A.8D, IC344A.8D, IC345A.8D, IC347A.8D, IC348A.8D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
- removed net RES0: IC246D.O, X2-4.KL
- removed net RES1: IC250C.O, X2-6.KL
- removed net RES2: IC260C.O, X2-8.KL
- removed net RES3: IC261C.O, X2-10.KL
- removed net RES4: IC262C.O, X2-12.KL
- removed net RES5: IC272C.O, X2-14.KL
- removed net RES6: IC273C.O, X2-16.KL
- removed net RES7: IC274C.O, X2-18.KL
- removed net RSEL0N: IC336A.G, IC362A.O
- removed net RSEL10N: IC346A.G
- removed net RSEL11N: IC347A.G, IC369C.O
- removed net RSEL12N: IC348A.G, IC369D.O
- removed net RSEL13N: IC349A.G, IC370A.O
- removed net RSEL14N: IC350A.G, IC370B.O
- removed net RSEL15N: IC351A.G, IC370C.O
- removed net RSEL1N: IC337A.G, IC362B.O
- removed net RSEL2N: IC338A.G, IC362C.O
- removed net RSEL3N: IC339A.G, IC362D.O
- removed net RSEL4N: IC340A.G, IC368A.O
- removed net RSEL5N: IC341A.G, IC368B.O
- removed net RSEL6N: IC342A.G, IC368C.O
- removed net RSEL7N: IC343A.G, IC368D.O
- removed net RSEL8N: IC344A.G, IC369A.O
- removed net RSEL9N: IC345A.G, IC369B.O
- removed net SIGN_REG: X2-26.KL
- removed net SUB_SEL_N: IC239B.O, IC243A.I1
- removed net VCC1: IC171P.VCC, IC172P.VCC, IC173P.VCC, IC174P.VCC, IC175P.VCC, IC176P.VCC, IC177P.VCC, IC178P.VCC, IC179P.VCC, IC180P.VCC, IC181P.VCC, IC182P.VCC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
- removed net VCC3: IC275P.VCC, IC276P.VCC, IC277P.VCC, IC278P.VCC, IC279P.VCC, IC280P.VCC, IC281P.VCC, IC282P.VCC, IC283P.VCC, IC284P.VCC, IC285P.VCC, IC286P.VCC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
- removed net Z_REG: X2-28.KL
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Other:
- note added: "Compare"
- note added: "PC_JMP_MUX"
- note removed: "PC"
- note removed: "Sign Extension Inverters"
